File: cryonano-nano-stage/buck-converter-1.kicad_sch (KiCad schematic)
At the start: 1 part

Commit message: sch updated
Parts:
- added PS3: B2415S-2WR3, symbol symbols:BxxxxS-2WR3
- PS1: renamed from PS2; Order No. (none) -> B2415S-1WR3; Unit Price 10 (none) -> 110
Connections:
- net +15V0OUT: now also PS3.6 (+VOUT)
- net +24V0IN: now also PS3.1 (+VIN)
- net 0V0IN: now also PS3.2 (GND)
- net 0V0OUT: now also PS3.4 (-VOUT)
Other:
- moved on the sheet: PS1
