File: cryonano-nano-stage/buck-converter-2.kicad_sch (KiCad schematic)
At the start: 1 part, among them U3 1ED3141MU12FXUMA1

Commit message: preliminary components added
Parts:
- removed U3: 1ED3141MU12FXUMA1, SOIC127P600X175-8N, symbol symbols:1ED3141MU12FXUMA1
- added PS1: HLK-B2405S-2WR3, HLKB2405S2WR3, symbol symbols:HLK-B2405S-2WR3
Changed lines of the file:
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@@
 	(generator_version "10.0")
 	(paper "A4")
+	(title_block
+		(rev "1.0.0")
+	)
+	(hierarchical_label "+5V0OUT"
+		(shape output)
+		(at 101.6 63.5 0)
+		(effects
+			(font
+				(size 1.27 1.27)
+			)
+			(justify left)
+		)
+	)
+	(hierarchical_label "+24V0IN"
+		(shape input)
+		(at 50.8 63.5 180)
+		(effects
+			(font
+				(size 1.27 1.27)
+			)
+			(justify right)
+		)
+	)
+	(hierarchical_label "0V0IN"
+		(shape input)
+		(at 50.8 68.58 180)
+		(effects
+			(font
+				(size 1.27 1.27)
+			)
+			(justify right)
+		)
+	)
+	(hierarchical_label "0V0OUT"
+		(shape output)
+		(at 101.6 68.58 0)
+		(effects
+			(font
+				(size 1.27 1.27)
+			)
+			(justify left)
+		)
+	)
 	(symbol
-		(lib_id "symbols:1ED3141MU12FXUMA1")
-		(at 101.6 101.6 0)
+		(lib_id "symbols:HLK-B2405S-2WR3")
+		(at 60.96 63.5 0)
 		(unit 1)
 		(body_style 1)
@@
 		(dnp no)
 		(fields_autoplaced yes)
-		(property "Reference" "U3"
-			(at 115.57 93.98 0)
-			(show_name no)
-			(do_not_autoplace no)
-			(effects
-				(font
-					(size 1.27 1.27)
-				)
-			)
-		)
-		(property "Value" "1ED3141MU12FXUMA1"
-			(at 115.57 96.52 0)
-			(show_name no)
-			(do_not_autoplace no)
-			(effects
-				(font
-					(size 1.27 1.27)
-				)
-			)
-		)
-		(property "Footprint" "SOIC127P600X175-8N"
-			(at 125.73 196.52 0)
-			(hide yes)
-			(show_name no)
-			(do_not_autoplace no)
-			(effects
-				(font
-					(size 1.27 1.27)
-				)
-				(justify left top)
-			)
-		)
-		(property "Datasheet" "https://www.mouser.in/datasheet/2/196/Infineon_1ED314xMU12F_DataSheet_v01_00_EN-3106223.pdf"
-			(at 125.73 296.52 0)
-			(hide yes)
-			(show_name no)
-			(do_not_autoplace no)
-			(effects
-				(font
-					(size 1.27 1.27)
-				)
-				(justify left top)
-			)
-		)
-		(property "Description" "Galvanically Isolated Gate Drivers ISOLATED DRIVER"
-			(at 101.6 101.6 0)
-			(hide yes)
-			(show_name no)
-			(do_not_autoplace no)
-			(effects
-				(font
-					(size 1.27 1.27)
-				)
-			)
-		)
-		(property "Height" "1.75"
-			(at 125.73 496.52 0)
-			(hide yes)
-			(show_name no)
-			(do_not_autoplace no)
-			(effects
-				(font
-					(size 1.27 1.27)
-				)
-				(justify left top)
-			)
-		)
-		(property "element14 Part Number" ""
-			(at 125.73 596.52 0)
-			(hide yes)
-			(show_name no)
-			(do_not_autoplace no)
-			(effects
-				(font
-					(size 1.27 1.27)
-				)
-				(justify left top)
-			)
-		)
-		(property "element14 Price/Stock" ""
-			(at 125.73 696.52 0)
-			(hide yes)
-			(show_name no)
-			(do_not_autoplace no)
-			(effects
-				(font
-					(size 1.27 1.27)
-				)
-				(justify left top)
-			)
-		)
-		(property "Manufacturer_Name" "Infineon"
-			(at 125.73 796.52 0)
-			(hide yes)
-			(show_name no)
-			(do_not_autoplace no)
-			(effects
-				(font
-					(size 1.27 1.27)
-				)
-				(justify left top)
-			)
-		)
-		(property "Manufacturer_Part_Number" "1ED3141MU12FXUMA1"
-			(at 125.73 896.52 0)
+		(property "Reference" "PS1"
+			(at 73.66 55.88 0)
+			(show_name no)
+			(do_not_autoplace no)
+			(effects
+				(font
+					(size 1.27 1.27)
+				)
+			)
+		)
+		(property "Value" "HLK-B2405S-2WR3"
+			(at 73.66 58.42 0)
+			(show_name no)
+			(do_not_autoplace no)
+			(effects
+				(font
+					(size 1.27 1.27)
+				)
+			)
+		)
+		(property "Footprint" "HLKB2405S2WR3"
+			(at 82.55 158.42 0)
+			(hide yes)
+			(show_name no)
+			(do_not_autoplace no)
+			(effects
+				(font
+					(size 1.27 1.27)
+				)
+				(justify left top)
+			)
+		)
+		(property "Datasheet" "https://datasheet.lcsc.com/lcsc/2206021745_HI-LINK-HLK-B2405S-2WR3_C3029164.pdf"
+			(at 82.55 258.42 0)
+			(hide yes)
+			(show_name no)
+			(do_not_autoplace no)
+			(effects
+				(font
+					(size 1.27 1.27)
+				)
+				(justify left top)
+			)
+		)
+		(property "Description" "5V 2400uF 400mA 21.6V~26.4V 1 Isolated Unregulated 2W DC-DC Short-Circuit Protection 86%~88% Plugin Power Modules ROHS"
+			(at 65.024 79.248 0)
+			(hide yes)
+			(show_name no)
+			(do_not_autoplace no)
+			(effects
+				(font
+					(size 1.27 1.27)
+				)
+			)
+		)
+		(property "Height" "10.25"
+			(at 82.55 458.42 0)
+			(hide yes)
+			(show_name no)
+			(do_not_autoplace no)
+			(effects
+				(font
+					(size 1.27 1.27)
+				)
+				(justify left top)
+			)
+		)
+		(property "Manufacturer_Name" "Hi-Link"
+			(at 82.55 558.42 0)
+			(hide yes)
+			(show_name no)
+			(do_not_autoplace no)
+			(effects
+				(font
+					(size 1.27 1.27)
+				)
+				(justify left top)
+			)
+		)
+		(property "Manufacturer_Part_Number" "HLK-B2405S-2WR3"
+			(at 82.55 658.42 0)
+			(hide yes)
+			(show_name no)
+			(do_not_autoplace no)
+			(effects
+				(font
+					(size 1.27 1.27)
+				)
+				(justify left top)
+			)
+		)
+		(property "Mouser Part Number" ""
+			(at 82.55 758.42 0)
+			(hide yes)
+			(show_name no)
+			(do_not_autoplace no)
+			(effects
+				(font
+					(size 1.27 1.27)
+				)
+				(justify left top)
+			)
+		)
+		(property "Mouser Price/Stock" ""
+			(at 82.55 858.42 0)
+			(hide yes)
+			(show_name no)
+			(do_not_autoplace no)
+			(effects
+				(font
+					(size 1.27 1.27)
+				)
+				(justify left top)
+			)
+		)
+		(property "Arrow Part Number" ""
+			(at 82.55 958.42 0)
+			(hide yes)
+			(show_name no)
+			(do_not_autoplace no)
+			(effects
+				(font
+					(size 1.27 1.27)
+				)
+				(justify left top)
+			)
+		)
+		(property "Arrow Price/Stock" ""
+			(at 82.55 1058.42 0)
 			(hide yes)
 			(show_name no)
@@
 		(pin "6"
 		)
-		(pin "5"
-		)
-		(pin "7"
-		)
 		(pin "1"
 		)
 		(pin "2"
 		)
-		(pin "3"
-		)
 		(pin "4"
-		)
-		(pin "8"
 		)
 		(instances
 			(project "cryonano-nano-stage"
-				(path "/549c6da5-71cb-4d9c-a0a2-c409a6f93509/37ffb213-c706-4fdf-aede-61f2739d8503/134546d9-2553-4cbc-b149-ff74fa29d06b"
-					(reference "U3")
+				(path "/549c6da5-71cb-4d9c-a0a2-c409a6f93509/0ae8b125-dbe2-44df-bbd5-11d3a39005e3/4b5b1cfb-c261-4252-ad9c-a17348397046"
+					(reference "PS1")
 					(unit 1)
 				)

Commit message: sch updated
Parts:
- removed PS1: HLK-B2405S-2WR3, HLKB2405S2WR3, symbol symbols:HLK-B2405S-2WR3
- added PS2: B2405S-1WR3, symbol symbols:BxxxxS-1WR3
- added PS4: B2405S-2WR3, symbol symbols:BxxxxS-2WR3
Connections:
- net +24V0IN: now also PS2.2 (+VIN), PS4.1 (+VIN)
- net +5V0OUT: now also PS2.4 (+VO), PS4.6 (+VOUT)
- net 0V0IN: now also PS2.1 (GND), PS4.2 (GND)
- net 0V0OUT: now also PS2.3 (-VO), PS4.4 (-VOUT)
