File: cryonano-nano-stage/cryonano-nano-stage.kicad_sch (KiCad schematic)
At the start: 0 parts

Commit message: few components listed
Other:
- added sheet ADC (adc.kicad_sch)
- added sheet Heater Controller (heater-controller.kicad_sch)
- added sheet Interface (interface.kicad_sch)
- added sheet MCU (mcu.kicad_sch)
- added sheet Power (power.kicad_sch)
Changed lines of the file:
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@@
 		(comment 8 "08-08-2026")
+	)
+	(sheet
+		(at 50.8 63.5)
+		(size 25.4 25.4)
+		(exclude_from_sim no)
+		(in_bom yes)
+		(on_board yes)
+		(dnp no)
+		(stroke
+			(width 0.1524)
+			(type solid)
+		)
+		(fill
+			(color 0 0 0 0)
+		)
+		(property "Sheetname" "Power"
+			(at 59.69 76.2 0)
+			(show_name no)
+			(do_not_autoplace no)
+			(effects
+				(font
+					(size 2.54 2.54)
+				)
+				(justify left bottom)
+			)
+		)
+		(property "Sheetfile" "power.kicad_sch"
+			(at 50.8 89.4846 0)
+			(hide yes)
+			(show_name no)
+			(do_not_autoplace no)
+			(effects
+				(font
+					(size 1.27 1.27)
+				)
+				(justify left top)
+			)
+		)
+		(instances
+			(project "cryonano-nano-stage"
+				(path "/549c6da5-71cb-4d9c-a0a2-c409a6f93509"
+					(page "2")
+				)
+			)
+		)
+	)
+	(sheet
+		(at 152.4 101.6)
+		(size 38.1 38.1)
+		(exclude_from_sim no)
+		(in_bom yes)
+		(on_board yes)
+		(dnp no)
+		(stroke
+			(width 0.1524)
+			(type solid)
+		)
+		(fill
+			(color 0 0 0 0)
+		)
+		(property "Sheetname" "Heater Controller"
+			(at 155.702 122.174 0)
+			(show_name no)
+			(do_not_autoplace no)
+			(effects
+				(font
+					(size 2.54 2.54)
+				)
+				(justify left bottom)
+			)
+		)
+		(property "Sheetfile" "heater-controller.kicad_sch"
+			(at 152.4 140.2846 0)
+			(hide yes)
+			(show_name no)
+			(do_not_autoplace no)
+			(effects
+				(font
+					(size 1.27 1.27)
+				)
+				(justify left top)
+			)
+		)
+		(instances
+			(project "cryonano-nano-stage"
+				(path "/549c6da5-71cb-4d9c-a0a2-c409a6f93509"
+					(page "6")
+				)
+			)
+		)
+	)
+	(sheet
+		(at 203.2 63.5)
+		(size 26.67 25.4)
+		(exclude_from_sim no)
+		(in_bom yes)
+		(on_board yes)
+		(dnp no)
+		(stroke
+			(width 0.1524)
+			(type solid)
+		)
+		(fill
+			(color 0 0 0 0)
+		)
+		(property "Sheetname" "Interface"
+			(at 212.852 74.93 0)
+			(show_name no)
+			(do_not_autoplace no)
+			(effects
+				(font
+					(size 2.54 2.54)
+				)
+				(justify left bottom)
+			)
+		)
+		(property "Sheetfile" "interface.kicad_sch"
+			(at 203.2 89.4846 0)
+			(hide yes)
+			(show_name no)
+			(do_not_autoplace no)
+			(effects
+				(font
+					(size 1.27 1.27)
+				)
+				(justify left top)
+			)
+		)
+		(instances
+			(project "cryonano-nano-stage"
+				(path "/549c6da5-71cb-4d9c-a0a2-c409a6f93509"
+					(page "5")
+				)
+			)
+		)
+	)
+	(sheet
+		(at 152.4 63.5)
+		(size 25.4 25.4)
+		(exclude_from_sim no)
+		(in_bom yes)
+		(on_board yes)
+		(dnp no)
+		(stroke
+			(width 0.1524)
+			(type solid)
+		)
+		(fill
+			(color 0 0 0 0)
+		)
+		(property "Sheetname" "ADC"
+			(at 164.084 76.962 0)
+			(show_name no)
+			(do_not_autoplace no)
+			(effects
+				(font
+					(size 2.54 2.54)
+				)
+				(justify left bottom)
+			)
+		)
+		(property "Sheetfile" "adc.kicad_sch"
+			(at 152.4 89.4846 0)
+			(hide yes)
+			(show_name no)
+			(do_not_autoplace no)
+			(effects
+				(font
+					(size 1.27 1.27)
+				)
+				(justify left top)
+			)
+		)
+		(instances
+			(project "cryonano-nano-stage"
+				(path "/549c6da5-71cb-4d9c-a0a2-c409a6f93509"
+					(page "3")
+				)
+			)
+		)
+	)
+	(sheet
+		(at 101.6 63.5)
+		(size 25.4 25.4)
+		(exclude_from_sim no)
+		(in_bom yes)
+		(on_board yes)
+		(dnp no)
+		(stroke
+			(width 0.1524)
+			(type solid)
+		)
+		(fill
+			(color 0 0 0 0)
+		)
+		(property "Sheetname" "MCU"
+			(at 114.554 76.454 0)
+			(show_name no)
+			(do_not_autoplace no)
+			(effects
+				(font
+					(size 2.54 2.54)
+				)
+				(justify left bottom)
+			)
+		)
+		(property "Sheetfile" "mcu.kicad_sch"
+			(at 101.6 89.4846 0)
+			(hide yes)
+			(show_name no)
+			(do_not_autoplace no)
+			(effects
+				(font
+					(size 1.27 1.27)
+				)
+				(justify left top)
+			)
+		)
+		(instances
+			(project "cryonano-nano-stage"
+				(path "/549c6da5-71cb-4d9c-a0a2-c409a6f93509"
+					(page "4")
+				)
+			)
+		)
 	)
 	(sheet_instances

Commit message: preliminary components added
Parts:
- added J1: Conn_01x03_Pin, symbol Connector:Conn_01x03_Pin
Connections:
- new net Earth: J1.3 (Pin_3)
- new net Power/+24V0IN: J1.1 (Pin_1)
- new net Power/0V0IN: J1.2 (Pin_2)
Other:
- added sheet USB (usb.kicad_sch)
- sheet Power ports: added +15V0_OUT_1, +24V0IN, +3V3_OUT_3, +5V0_OUT_2, 0V0IN, 0V0_OUT_1, 0V0_OUT_2, 0V0_OUT_3; removed none

Commit message: sch updated
Other:
- sheet MCU ports: added +3V3IN, +5V0IN, 0V0IN, CLKADC, DE/~{RE}, DM, DP; removed none
- sheet Power ports: added none; removed 0V0_OUT_3
- sheet USB ports: added DM; removed DN
Changed lines of the file:
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@@
+		)
+	)
+	(wire
+		(pts
+			(xy 124.46 101.6) (xy 124.46 111.76)
+		)
+		(stroke
+			(width 0)
+			(type default)
+		)
+	)
+	(wire
+		(pts
+			(xy 121.92 101.6) (xy 121.92 111.76)
+		)
+		(stroke
+			(width 0)
+			(type default)
 		)
 	)
@@
 			)
 		)
+		(property "Allied Price/Stock" ""
+			(at 25.4 83.82 0)
+			(hide yes)
+			(show_name no)
+			(do_not_autoplace no)
+			(effects
+				(font
+					(size 1.27 1.27)
+				)
+			)
+		)
+		(property "Allied_Number" ""
+			(at 25.4 83.82 0)
+			(hide yes)
+			(show_name no)
+			(do_not_autoplace no)
+			(effects
+				(font
+					(size 1.27 1.27)
+				)
+			)
+		)
+		(property "MCWR08X12R0FTL " ""
+			(at 25.4 83.82 0)
+			(hide yes)
+			(show_name no)
+			(do_not_autoplace no)
+			(effects
+				(font
+					(size 1.27 1.27)
+				)
+			)
+		)
+		(property "RS Part Number" ""
+			(at 25.4 83.82 0)
+			(hide yes)
+			(show_name no)
+			(do_not_autoplace no)
+			(effects
+				(font
+					(size 1.27 1.27)
+				)
+			)
+		)
+		(property "RS Price/Stock" ""
+			(at 25.4 83.82 0)
+			(hide yes)
+			(show_name no)
+			(do_not_autoplace no)
+			(effects
+				(font
+					(size 1.27 1.27)
+				)
+			)
+		)
 		(pin "3"
 		)
@@
 		(on_board yes)
 		(dnp no)
+		(fields_autoplaced yes)
 		(stroke
 			(width 0.1524)
@@
 		)
 		(property "Sheetname" "Power"
-			(at 49.784 84.582 0)
+			(at 38.1 62.1534 0)
 			(show_name no)
 			(do_not_autoplace no)
@@
 		)
 		(property "Sheetfile" "power.kicad_sch"
-			(at 38.1 89.4846 0)
+			(at 38.1 102.1846 0)
 			(hide yes)
 			(show_name no)
@@
 		(pin "0V0_OUT_2" output
 			(at 63.5 93.98 0)
-			(effects
-				(font
-					(size 1.27 1.27)
-				)
-				(justify right)
-			)
-		)
-		(pin "0V0_OUT_3" output
-			(at 63.5 96.52 0)
 			(effects
 				(font
@@
 			)
 		)
-		(pin "DN" input
-			(at 124.46 111.76 90)
-			(effects
-				(font
-					(size 1.27 1.27)
-				)
-				(justify right)
-			)
-		)
 		(pin "DP" input
 			(at 121.92 111.76 90)
+			(effects
+				(font
+					(size 1.27 1.27)
+				)
+				(justify right)
+			)
+		)
+		(pin "DM" input
+			(at 124.46 111.76 90)
 			(effects
 				(font
@@
 			)
 		)
+		(pin "+3V3IN" input
+			(at 106.68 63.5 90)
+			(effects
+				(font
+					(size 1.27 1.27)
+				)
+				(justify right)
+			)
+		)
+		(pin "+5V0IN" input
+			(at 104.14 63.5 90)
+			(effects
+				(font
+					(size 1.27 1.27)
+				)
+				(justify right)
+			)
+		)
+		(pin "0V0IN" input
+			(at 109.22 63.5 90)
+			(effects
+				(font
+					(size 1.27 1.27)
+				)
+				(justify right)
+			)
+		)
+		(pin "CLKADC" output
+			(at 127 69.85 0)
+			(effects
+				(font
+					(size 1.27 1.27)
+				)
+				(justify right)
+			)
+		)
+		(pin "DE{slash}~{RE}" output
+			(at 127 88.9 0)
+			(effects
+				(font
+					(size 1.27 1.27)
+				)
+				(justify right)
+			)
+		)
+		(pin "DM" bidirectional
+			(at 124.46 101.6 270)
+			(effects
+				(font
+					(size 1.27 1.27)
+				)
+				(justify left)
+			)
+		)
+		(pin "DP" bidirectional
+			(at 121.92 101.6 270)
+			(effects
+				(font
+					(size 1.27 1.27)
+				)
+				(justify left)
+			)
+		)

Commit message: partially populated
Parts:
- added H1, H2, H3, H4, H5, H6: MountingHole, footprints:MountingHole_3.7mm_Pad_Small, symbol Mechanical:MountingHole

Commit message: sch improved
Parts:
- removed H1, H2, H3, H4, H5, H6: MountingHole, footprints:MountingHole_3.7mm_Pad_Small, symbol Mechanical:MountingHole
- removed J1: Conn_01x03_Pin, symbol Connector:Conn_01x03_Pin
Other:
- removed sheet ADC
- removed sheet Heater Controller
- removed sheet Interface
- removed sheet MCU
- removed sheet Power
- removed sheet USB
- added sheet Block Diagram (block-diagram.kicad_sch)
- note added: "Brief: Two bridges can be controlled independently by the Microcontroller. Two RTD interface is implemented to measure temperature using Wheatstone bridge-balancing principle. Bridge resistances shall be adjusted according to the application requirement."
- note added: "Title: Schematic for heater control and temperature monitoring of nano-stage"

Commit message: sch improved
Other:
- note added: "Custom rules"
Changed lines of the file:
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@@
 		(effects
 			(font
-				(size 2.54 2.54)
+				(size 2.032 2.032)
 				(thickness 0.3175)
 			)
 			(justify left)
+		)
+	)
+	(text "Custom rules"
+		(exclude_from_sim no)
+		(at 143.764 158.75 0)
+		(effects
+			(font
+				(size 5.08 5.08)
+			)
 		)
 	)
@@
 			(font
 				(size 2.54 2.54)
-				(thickness 0.508)
-				(bold yes)
+				(thickness 0.1588)
 			)
 		)
@@
 				(font
 					(size 2.54 2.54)
-					(thickness 0.508)
-					(bold yes)
+					(thickness 0.1588)
 				)
 				(justify left bottom)
@@
 			(effects
 				(font
-					(size 2.54 2.54)
+					(size 1.27 1.27)
+					(thickness 0.1588)
 				)
 				(justify left top)
