File: cryonano-nano-stage/mcu-gpio-a-b-c.kicad_sch (KiCad schematic)
At the start: 1 part, among them U11 STM32H753ZITx

Commit message: sch improved
Parts:
- added C16, C17: 100n, Capacitor_SMD:C_0603_1608Metric, symbol Device:C_Small
- added C33, C34, C36, C37: 22pF, Capacitor_SMD:C_0603_1608Metric, symbol Device:C_Small
- added D1: PESD3V3S1UL, Diode_SMD:D_SOD-882, symbol Diode:PESD3V3S1UL
- added R35: 470R, Resistor_SMD:R_0603_1608Metric, symbol Device:R_Small
- added R36, R38, R86: 10k, Resistor_SMD:R_0603_1608Metric, symbol Device:R_Small
- added SW1: BOOT, Button_Switch_THT:SW_PUSH_6mm, symbol Switch:SW_Push
- added SW2: RESET, Button_Switch_THT:SW_PUSH_6mm, symbol Switch:SW_Push
- added Y2, Y4: 12.0MHz, Crystal:Crystal_SMD_3215-2Pin_3.2x1.5mm, symbol Device:Crystal
Connections:
- net PA8: now reaches U11.100 (PA8)
- net PA9: now reaches U11.101 (PA9)
- net PA10: now reaches U11.102 (PA10)
- net PA11: now reaches U11.103 (PA11)
- net PA12: now reaches U11.104 (PA12)
- net PA13: now reaches U11.105 (PA13)
- net PA14: now reaches U11.109 (PA14)
- net PA15: now reaches U11.110 (PA15)
- net PC10: now reaches U11.111 (PC10)
- net PC11: now reaches U11.112 (PC11)
- net PC12: now reaches U11.113 (PC12)
- net PB3: now reaches U11.133 (PB3)
- net PB4: now reaches U11.134 (PB4)
- net PB5: now reaches U11.135 (PB5)
- net PB6: now reaches U11.136 (PB6)
- net PB7: now reaches U11.137 (PB7)
- net BOOT0: now reaches U11.138 (BOOT0)
- net BOOT0: now also C16.1, R36.1, SW1.2
- net PB8: now reaches U11.139 (PB8)
- net PB9: now reaches U11.140 (PB9)
- net PDR_ON: now reaches U11.143 (PDR_ON)
- net PDR_ON: now also R38.2, R86.1
- net RCC_OSC_IN: now reaches U11.23 (PH0)
- net RCC_OSC_IN: now also C33.1, Y4.2
- net RCC_OSC_OUT: now reaches U11.24 (PH1)
- net RCC_OSC_OUT: now also C34.1, Y4.1
- net NRST: now reaches U11.25 (NRST)
- net NRST: now also C17.1, D1.1 (K), SW2.1
- net PC0: now reaches U11.26 (PC0)
- net PC1: now reaches U11.27 (PC1)
- net PC2: now reaches U11.28 (PC2_C)
- net PC3: now reaches U11.29 (PC3_C)
- net PA0: now reaches U11.34 (PA0)
- net PA1: now reaches U11.35 (PA1)
- net PA2: now reaches U11.36 (PA2)
- net PA3: now reaches U11.37 (PA3)
- net PA4: now reaches U11.40 (PA4)
- net PA5: now reaches U11.41 (PA5)
- net PA6: now reaches U11.42 (PA6)
- net PA7: now reaches U11.43 (PA7)
- net PC4: now reaches U11.44 (PC4)
- net PC5: now reaches U11.45 (PC5)
- net PB0: now reaches U11.46 (PB0)
- net PB1: now reaches U11.47 (PB1)
- net PB2: now reaches U11.48 (PB2)
- net PB10: now reaches U11.69 (PB10)
- net PC13: now reaches U11.7 (PC13)
- net PB11: now reaches U11.70 (PB11)
- net PB12: now reaches U11.73 (PB12)
- net PB13: now reaches U11.74 (PB13)
- net PB14: now reaches U11.75 (PB14)
- net PB15: now reaches U11.76 (PB15)
- net RCC_OSC32_IN: now reaches U11.8 (PC14)
- net RCC_OSC32_IN: now also C36.1, Y2.2
- net RCC_OSC32_OUT: now reaches U11.9 (PC15)
- net RCC_OSC32_OUT: now also C37.1, Y2.1
- net PC6: now reaches U11.96 (PC6)
- net PC7: now reaches U11.97 (PC7)
- net PC8: now reaches U11.98 (PC8)
- net PC9: now reaches U11.99 (PC9)
- new net: R35.2, SW1.1
- new net VDD: R35.1, R38.1
- new net VSS: C16.2, C17.2, C33.2, C34.2, C36.2, C37.2, D1.2 (A), R36.2, R86.2, SW2.2
Other:
- note added: "BOOT memory selection."
- note added: "RESET"
- moved on the sheet: U11A
