File: cryonano-nano-stage/mcu-gpio-d-e-f-g.kicad_sch (KiCad schematic)
At the start: 1 part, among them U11 STM32H753ZITx

Commit message: sch improved
Connections:
- net PE2: now reaches U11.1 (PE2)
- net PF0: now reaches U11.10 (PF0)
- net PF1: now reaches U11.11 (PF1)
- net PD0: now reaches U11.114 (PD0)
- net PD1: now reaches U11.115 (PD1)
- net PD2: now reaches U11.116 (PD2)
- net PD3: now reaches U11.117 (PD3)
- net PD4: now reaches U11.118 (PD4)
- net PD5: now reaches U11.119 (PD5)
- net PF2: now reaches U11.12 (PF2)
- net PD6: now reaches U11.122 (PD6)
- net PD7: now reaches U11.123 (PD7)
- net PG9: now reaches U11.124 (PG9)
- net PG10: now reaches U11.125 (PG10)
- net PG11: now reaches U11.126 (PG11)
- net PG12: now reaches U11.127 (PG12)
- net PG13: now reaches U11.128 (PG13)
- net PG14: now reaches U11.129 (PG14)
- net PF3: now reaches U11.13 (PF3)
- net PG15: now reaches U11.132 (PG15)
- net PF4: now reaches U11.14 (PF4)
- net PE0: now reaches U11.141 (PE0)
- net PE1: now reaches U11.142 (PE1)
- net PF5: now reaches U11.15 (PF5)
- net PF6: now reaches U11.18 (PF6)
- net PF7: now reaches U11.19 (PF7)
- net PE3: now reaches U11.2 (PE3)
- net PF8: now reaches U11.20 (PF8)
- net PF9: now reaches U11.21 (PF9)
- net PF10: now reaches U11.22 (PF10)
- net PE4: now reaches U11.3 (PE4)
- net PE5: now reaches U11.4 (PE5)
- net PF11: now reaches U11.49 (PF11)
- net PE6: now reaches U11.5 (PE6)
- net PF12: now reaches U11.50 (PF12)
- net PF13: now reaches U11.53 (PF13)
- net PF14: now reaches U11.54 (PF14)
- net PF15: now reaches U11.55 (PF15)
- net PG0: now reaches U11.56 (PG0)
- net PG1: now reaches U11.57 (PG1)
- net PE7: now reaches U11.58 (PE7)
- net PE8: now reaches U11.59 (PE8)
- net PE9: now reaches U11.60 (PE9)
- net PE10: now reaches U11.63 (PE10)
- net PE11: now reaches U11.64 (PE11)
- net PE12: now reaches U11.65 (PE12)
- net PE13: now reaches U11.66 (PE13)
- net PE14: now reaches U11.67 (PE14)
- net PE15: now reaches U11.68 (PE15)
- net PD8: now reaches U11.77 (PD8)
- net PD9: now reaches U11.78 (PD9)
- net PD10: now reaches U11.79 (PD10)
- net PD11: now reaches U11.80 (PD11)
- net PD12: now reaches U11.81 (PD12)
- net PD13: now reaches U11.82 (PD13)
- net PD14: now reaches U11.85 (PD14)
- net PD15: now reaches U11.86 (PD15)
- net PG2: now reaches U11.87 (PG2)
- net PG3: now reaches U11.88 (PG3)
- net PG4: now reaches U11.89 (PG4)
- net PG5: now reaches U11.90 (PG5)
- net PG6: now reaches U11.91 (PG6)
- net PG7: now reaches U11.92 (PG7)
- net PG8: now reaches U11.93 (PG8)
