File: cryonano-nano-stage/cryonano-nano-stage.kicad_pcb (KiCad board)
At the start: 2 copper layers, 47 parts, among them J4 10118194-0001LF, J8 Conn_ST_STDC14, Q1 PMV100EPAR, SW1 ~{RESET}, SW2 BOOT0, U10 ECMF02-2AMX6, U3 1ED3141MU12FXUMA1, U4 AP7363-33D-13, U5 STM32L412CBT6P

Commit message: sch updated
Parts:
- removed C5, C7: 0.1uF, Capacitor_SMD:C_0603_1608Metric
- removed R11, R8: 47k, Resistor_SMD:R_0603_1608Metric
- removed R29, R30, R31, R32, R33, R34: 22R, Resistor_SMD:R_0603_1608Metric
- removed R5: 10k, Resistor_SMD:R_0603_1608Metric
- removed R9: 1k, Resistor_SMD:R_0603_1608Metric
- removed U5: STM32L412CBT6P, Package_QFP:LQFP-32_7x7mm_P0.8mm
- added C16: 0.1uF, Capacitor_SMD:C_0603_1608Metric, F.Cu at (122.4, 117.8)
- added C17: 0.1uF, Capacitor_SMD:C_0603_1608Metric, F.Cu at (122.4, 120.3)
- added R36: 10k, Resistor_SMD:R_0603_1608Metric, F.Cu at (122.4, 122.8)
- added R38: 10k, Resistor_SMD:R_0603_1608Metric, F.Cu at (122.4, 125.3)
- added U1: AD7124-8BCPZ-RL7, SamacSys_Parts:QFN50P500X500X80-33N-D, F.Cu at (112.5, 133.7)
- added U2: STM32L412CxTx, SamacSys_Parts:QFP50P900X900X160-48N, F.Cu at (105.4, 101.3)
- PS1: value HLK-B2405S-2WR3 -> B2415S-1WR3
- R35: value 47k -> 470R
- SW1: value ~{RESET} -> BOOT
- SW2: value BOOT0 -> RESET
- moved U10 47.0 mm to (104.7, 88.9), turned to 90 degrees
- moved J4 5.11 mm to (104.1, 82.3), turned to 180 degrees
Connections:
- net /Power/0V0_OUT_2 renamed /Power/Buck converter 2/MOUT
- net /Power/Buck converter 2/+5V0OUT renamed /Power/Buck converter 2/+VOUT
- J8 pad 12: /MCU/T_NRST -> /MCU/NRST
- J8 pad 13: /MCU/T_VCP_RX -> /MCU/LOG_RX
- J8 pad 14: /MCU/T_VCP_TX -> /MCU/LOG_TX
- J8 pad 4: /MCU/T_JTMS/T_SWDIO  -> /MCU/SWDIO
- J8 pad 6: /MCU/T_JCLK/T_SWCLK -> /MCU/SWCLK
- J8 pad 8: /MCU/T_JTDO/T_SWO -> /MCU/SWO
- PS1 pad 1: unconnected-(PS1-+VIN-Pad1) -> /Power/0V0
- PS1 pad 2: unconnected-(PS1--VIN-Pad2) -> /Power/+24V0
- PS1 pad 4: unconnected-(PS1--VOUT-Pad4) -> /Power/Buck converter 1/+VOUT
- PS1 pad 6: unconnected-(PS1-+VOUT-Pad6) -> (no net)
- R35 pad 1: /MCU/STATUS_RGB_SDA -> /MCU/+3V3V
- R35 pad 2: /MCU/+3V3V -> Net-(R35-Pad2)
- SW1 pad 1: /MCU/T_NRST -> Net-(R35-Pad2)
- SW1 pad 2: GND -> /MCU/BOOT0
- SW2 pad 1: /MCU/BOOT0 -> /MCU/NRST
- SW2 pad 2: Net-(R9-Pad2) -> GND
- U10 pad 1: /USB/USB_P -> /MCU/USB_D+
- U10 pad 2: /USB/USB_N -> /MCU/USB_D-

Commit message: partially populated
Parts:
- removed PS1: B2415S-1WR3, SamacSys_Parts:HLKB2405S2WR3
- removed SW1: BOOT, Button_Switch_SMD:SW_Tactile_SPST_NO_Straight_CK_PTS636Sx25SMTRLFS
- removed SW2: RESET, Button_Switch_SMD:SW_Tactile_SPST_NO_Straight_CK_PTS636Sx25SMTRLFS
- added H1: MountingHole, footprints:MountingHole_3.7mm_Pad_Small, F.Cu at (105.0, 120.0)
- added H2: MountingHole, footprints:MountingHole_3.7mm_Pad_Small, F.Cu at (140.0, 120.0)
- added H3: MountingHole, footprints:MountingHole_3.7mm_Pad_Small, F.Cu at (175.0, 120.0)
- added H4: MountingHole, footprints:MountingHole_3.7mm_Pad_Small, F.Cu at (175.0, 90.0)
- added H5: MountingHole, footprints:MountingHole_3.7mm_Pad_Small, F.Cu at (140.0, 90.0)
- added H6: MountingHole, footprints:MountingHole_3.7mm_Pad_Small, F.Cu at (105.0, 90.0)
- moved C14 57.3 mm to (166.4, 81.5)
- moved C15 57.3 mm to (166.4, 84.0)
- moved FB3 56.1 mm to (166.4, 94.1)
- moved C64 56.1 mm to (166.4, 91.6)
- moved C17 53.9 mm to (166.4, 89.0)
- moved C16 53.9 mm to (166.4, 86.5)
- moved J8 50.6 mm to (135.3, 108.1), turned to 90 degrees
- moved R36 50.0 mm to (166.4, 99.1)
- moved R38 50.0 mm to (166.4, 101.6)
- moved U1 47.9 mm to (153.9, 109.5)
- moved R35 47.3 mm to (166.4, 96.6)
- moved F1 45.7 mm to (108.3, 112.6)
- moved D2 45.5 mm to (108.5, 102.4)
- moved D4 45.5 mm to (108.5, 105.3)
- moved U4 41.5 mm to (107.3, 98.4)
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Routing:
- net GND: track 0.00 -> 27.4 mm
Other:
- board outline added: 80 x 40 mm
- copper layers 2 -> 4

Commit message: sch improved
Parts:
- removed C10: 100n, Capacitor_SMD:C_0603_1608Metric
- removed FB1, FB2: BLM21PG221SN1D, Inductor_SMD:L_0805_2012Metric
- removed J4: 10118194-0001LF, footprints:101181940001LF
- added C12: 10u, Capacitor_SMD:C_0805_2012Metric, F.Cu at (250.6, 122.8)
- added C13: 10u, Capacitor_SMD:C_0805_2012Metric, F.Cu at (123.8, 45.4)
- added C18: 100n, Capacitor_SMD:C_0603_1608Metric, F.Cu at (241.2, 115.2)
- added C19: 100n, Capacitor_SMD:C_0603_1608Metric, F.Cu at (110.2, 32.6)
- added C2: 100n, Capacitor_SMD:C_0603_1608Metric, F.Cu at (265.0, 88.9)
- added C22: 100n, Capacitor_SMD:C_0603_1608Metric, F.Cu at (110.2, 35.1)
- added C23: 100n, Capacitor_SMD:C_0603_1608Metric, F.Cu at (110.2, 37.6)
- added C24: 5.6p, Capacitor_SMD:C_0603_1608Metric, F.Cu at (110.2, 40.1)
- added C25: 5.6p, Capacitor_SMD:C_0603_1608Metric, F.Cu at (110.2, 42.6)
- added C26: 470p, Capacitor_SMD:C_0603_1608Metric, F.Cu at (114.3, 32.6)
- added C27: 1u, Capacitor_SMD:C_0603_1608Metric, F.Cu at (241.2, 117.8)
- added C28: 1u, Capacitor_SMD:C_0603_1608Metric, F.Cu at (241.2, 120.3)
- added C29: 1u, Capacitor_SMD:C_0603_1608Metric, F.Cu at (241.2, 81.1)
- added C30: 1u, Capacitor_SMD:C_0603_1608Metric, F.Cu at (114.3, 35.1)
- added C31: 100n, Capacitor_SMD:C_0603_1608Metric, F.Cu at (110.8, 14.5)
- added C32: 1u, Capacitor_SMD:C_0603_1608Metric, F.Cu at (241.2, 83.6)
- added C33: 1u, Capacitor_SMD:C_0603_1608Metric, F.Cu at (241.2, 86.1)
- added C34: 1u, Capacitor_SMD:C_0603_1608Metric, F.Cu at (241.2, 88.6)
- added C35: 1n, Capacitor_SMD:C_0603_1608Metric, F.Cu at (110.8, 17.0)
- added C38: 100n, Capacitor_SMD:C_0603_1608Metric, F.Cu at (110.8, 19.5)
- added C65: 1n, Capacitor_THT:C_Disc_D9.0mm_W5.0mm_P10.00mm, F.Cu at (205.1, 135.9)
- added C66: 100n, Capacitor_SMD:C_0603_1608Metric, F.Cu at (241.2, 122.8)
- added C67: 100n, Capacitor_SMD:C_0603_1608Metric, F.Cu at (241.2, 91.1)
- added C68: 10u, Capacitor_SMD:C_0805_2012Metric, F.Cu at (253.4, 90.6)
- added C69: 100n, Capacitor_SMD:C_0603_1608Metric, F.Cu at (209.4, 34.3)
- added D8: PESD12VL1BA, Diode_SMD:D_SOD-323F, F.Cu at (205.5, 144.7)
- added FB4: MH1608, Inductor_SMD:L_0603_1608Metric, F.Cu at (114.3, 37.6)
- added FB5: MH1608, Inductor_SMD:L_0603_1608Metric, F.Cu at (238.8, 103.1)
- added FB7: BLM21PG221SN1D, Inductor_SMD:L_0805_2012Metric, F.Cu at (260.7, 89.0)
- added FB8: BLM21PG221SN1D, Inductor_SMD:L_0805_2012Metric, F.Cu at (260.7, 91.8)
- added J1: 24VDC IN, footprints:B3BXHAMLFSN, F.Cu at (219.3, 77.3)
- added J2: JST-B2B-XH-AM, SamacSys_Parts:B2BXHAMLFSN, F.Cu at (229.1, 76.7)
- added J3: JST-B2B-XH-AM, SamacSys_Parts:B2BXHAMLFSN, F.Cu at (229.1, 84.3)
- added J5: JST-B3B-XH-AM, footprints:B3BXHAMLFSN, F.Cu at (219.3, 86.2)
- added J6: RJ45_Hanrun_HR911105A_Horizontal, footprints:RJ45_Hanrun_HR911105A_Horizontal, F.Cu at (137.8, 26.2)
- added J7: 10118194-0001LF, footprints:101181940001LF, F.Cu at (264.4, 84.9)
- added PS1: B2415S-1WR3, SamacSys_Parts:HLKB2405S2WR3, F.Cu at (258.9, 113.9)
- added PS2: B2405S-1WR3, SamacSys_Parts:HLKB2405S2WR3, F.Cu at (258.9, 101.7)
- added R26: 1M, Resistor_THT:R_Axial_DIN0207_L6.3mm_D2.5mm_P10.16mm_Horizontal, F.Cu at (204.9, 141.2)
- added R27: 10k, Resistor_SMD:R_0603_1608Metric, F.Cu at (201.4, 60.7)
- added R37: 1k2, Resistor_SMD:R_0603_1608Metric, F.Cu at (201.4, 63.2)
- added R39: 1k2, Resistor_SMD:R_0603_1608Metric, F.Cu at (201.4, 65.7)
- added R40: 22R, Resistor_SMD:R_0603_1608Metric, F.Cu at (241.2, 108.2)
- added R41: 10k, Resistor_SMD:R_0603_1608Metric, F.Cu at (241.2, 93.7)
- added R42: 10k, Resistor_SMD:R_0603_1608Metric, F.Cu at (241.2, 96.2)
- added R43: 10k, Resistor_SMD:R_0603_1608Metric, F.Cu at (245.2, 81.1)
- added R44: 10k, Resistor_SMD:R_0603_1608Metric, F.Cu at (245.2, 83.6)
- added R45: 0R, Resistor_SMD:R_0603_1608Metric, F.Cu at (245.2, 86.1)
- added R46: 0R, Resistor_SMD:R_0603_1608Metric, F.Cu at (245.2, 88.6)
- added R47: 0R, Resistor_SMD:R_0603_1608Metric, F.Cu at (245.2, 91.1)
- added R48: 0R, Resistor_SMD:R_0603_1608Metric, F.Cu at (245.2, 93.7)
- added R49: 0R, Resistor_SMD:R_0603_1608Metric, F.Cu at (245.2, 96.2)
- added R50: 0R, Resistor_SMD:R_0603_1608Metric, F.Cu at (249.2, 81.1)
- added R51: 10k, Resistor_SMD:R_0603_1608Metric, F.Cu at (249.2, 83.6)
- added R52: 0R, Resistor_SMD:R_0603_1608Metric, F.Cu at (249.2, 86.1)
- added R53: 10k, Resistor_SMD:R_0603_1608Metric, F.Cu at (249.2, 88.6)
- added R54: 0R, Resistor_SMD:R_0603_1608Metric, F.Cu at (249.2, 91.1)
- added R55: 10k, Resistor_SMD:R_0603_1608Metric, F.Cu at (249.2, 93.7)
- added R56: 10k, Resistor_SMD:R_0603_1608Metric, F.Cu at (249.2, 96.2)
- added R57: 10k, Resistor_SMD:R_0603_1608Metric, F.Cu at (114.3, 40.1)
- added R58: 10k, Resistor_SMD:R_0603_1608Metric, F.Cu at (114.3, 42.6)
- added R59: 10k, Resistor_SMD:R_0603_1608Metric, F.Cu at (118.3, 32.6)
- added R60: 1k5, Resistor_SMD:R_0603_1608Metric, F.Cu at (118.3, 35.1)
- added R61: 10k, Resistor_SMD:R_0603_1608Metric, F.Cu at (118.3, 37.6)
- added R62: 33R, Resistor_SMD:R_0603_1608Metric, F.Cu at (118.3, 40.1)
- added R63: 33R, Resistor_SMD:R_0603_1608Metric, F.Cu at (118.3, 42.6)
- added R64: 10k, Resistor_SMD:R_0603_1608Metric, F.Cu at (122.3, 32.6)
- added R65: 33R, Resistor_SMD:R_0603_1608Metric, F.Cu at (122.3, 35.1)
- added R66: 33R, Resistor_SMD:R_0603_1608Metric, F.Cu at (122.3, 37.6)
- added R67: 0R, Resistor_SMD:R_0603_1608Metric, F.Cu at (122.3, 40.1)
- added R68: 0R, Resistor_SMD:R_0603_1608Metric, F.Cu at (122.3, 42.6)
- added R69: 49.9R, Resistor_SMD:R_0603_1608Metric, F.Cu at (110.8, 22.0)
- added R70: 49.9R, Resistor_SMD:R_0603_1608Metric, F.Cu at (110.8, 24.5)
- added R71: 49.9R, Resistor_SMD:R_0603_1608Metric, F.Cu at (114.8, 14.5)
- added R72: 49.9R, Resistor_SMD:R_0603_1608Metric, F.Cu at (114.8, 17.0)
- added R73: 270R, Resistor_SMD:R_0603_1608Metric, F.Cu at (114.8, 19.5)
- added R74: 270R, Resistor_SMD:R_0603_1608Metric, F.Cu at (114.8, 22.0)
- added R75: 12k1, Resistor_SMD:R_0603_1608Metric, F.Cu at (114.8, 24.5)
- added R76: 4k7, Resistor_SMD:R_0603_1608Metric, F.Cu at (209.4, 36.8)
- added R77: 4k7, Resistor_SMD:R_0603_1608Metric, F.Cu at (209.4, 39.3)
- added R78: 4k7, Resistor_SMD:R_0603_1608Metric, F.Cu at (209.4, 41.8)
- added R79: 4k7, Resistor_SMD:R_0603_1608Metric, F.Cu at (209.4, 44.3)
- added R80: 4k7, Resistor_SMD:R_0603_1608Metric, F.Cu at (209.4, 46.8)
- added R81: 4k7, Resistor_SMD:R_0603_1608Metric, F.Cu at (213.4, 34.3)
- added R82: 4k7, Resistor_SMD:R_0603_1608Metric, F.Cu at (213.4, 36.8)
- added R83: 4k7, Resistor_SMD:R_0603_1608Metric, F.Cu at (213.4, 39.3)
- added R84: 4k7, Resistor_SMD:R_0603_1608Metric, F.Cu at (213.4, 41.8)
- added R85: 4k7, Resistor_SMD:R_0603_1608Metric, F.Cu at (213.4, 44.3)
- added SW1: BOOT, Button_Switch_THT:SW_PUSH_6mm, F.Cu at (246.1, 52.5)
- added SW2: RESET, Button_Switch_THT:SW_PUSH_6mm, F.Cu at (246.1, 61.1)
- added U5: ECMF02-2AMX6, Package_DFN_QFN:ST_UQFN-6L_1.5x1.7mm_P0.5mm, F.Cu at (268.9, 89.3)
- added U6: LP5907MFX-3.3_NOPB, SamacSys_Parts:SOT95P280X145-5N, F.Cu at (245.8, 123.6)
- added U7: LP5907MFX-3.3_NOPB, SamacSys_Parts:SOT95P280X145-5N, F.Cu at (253.8, 82.2)
- added U8: LP5907MFX-3.3_NOPB, SamacSys_Parts:SOT95P280X145-5N, F.Cu at (253.8, 86.8)
- added U9: USBLC6-4SC6, Package_TO_SOT_SMD:SOT-23-6, F.Cu at (143.6, 34.5)
- added Y3: 25.0MHz, Crystal:Crystal_SMD_3225-4Pin_3.2x2.5mm_HandSoldering, F.Cu at (118.2, 46.8)
- added Z2: MM1W18, Diode_SMD:D_SOD-123, F.Cu at (213.2, 121.3)
- C1: value 100uF -> 100u
- C11: value 10uF -> 10u
- C14, C15, C16, C17, C64: value 0.1uF -> 100n
- C3: value 10uF -> 10u; footprint Capacitor_SMD:C_1210_3225Metric -> Capacitor_SMD:C_1206_3216Metric
- U10: value ECMF02-2AMX6 -> LAN8742A; footprint Package_DFN_QFN:ST_UQFN-6L_1.5x1.7mm_P0.5mm -> Package_DFN_QFN:VQFN-24-1EP_4x4mm_P0.5mm_EP2.5x2.5mm_ThermalVias
- moved J8 138.1 mm to (267.3, 67.7), turned to 0 degrees
- moved C11 136.9 mm to (272.9, 67.5)
- moved U2 136.8 mm to (271.0, 60.2), turned to 0 degrees
- moved H6 129.6 mm to (232.7, 67.9)
- moved H1 125.6 mm to (214.8, 59.0)
- moved U3 116.9 mm to (247.4, 102.7)
- moved C1 107.0 mm to (221.4, 96.9)
- moved F1 107.0 mm to (215.2, 116.2)
- moved FL2 107.0 mm to (222.5, 111.8)
- moved Q1 107.0 mm to (215.6, 112.7)
- moved D11 107.0 mm to (231.1, 110.8)
- moved GD1 107.0 mm to (230.0, 115.6)
- moved MOV1 107.0 mm to (221.0, 103.7)
- moved R1 107.0 mm to (229.9, 100.1)
- moved TP1 107.0 mm to (211.8, 106.0)
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Connections:
- net /MCU/+3V3V renamed /Block Diagram/Controller/+3V3V
- net /MCU/BOOT0 renamed /Block Diagram/Controller/BOOT0
- net /MCU/LOG_RX renamed /Block Diagram/Controller/LOG_RX
- net /MCU/LOG_TX renamed /Block Diagram/Controller/LOG_TX
- net /MCU/NRST renamed /Block Diagram/Controller/NRST
- net /MCU/SWCLK renamed /Block Diagram/Controller/SWCLK
- net /MCU/SWDIO renamed /Block Diagram/Controller/SWDIO
- net /MCU/SWO renamed /Block Diagram/Controller/SWO
- net /MCU/VBAT renamed /Block Diagram/Controller/VBAT
- net /MCU/VDDA renamed /Block Diagram/Controller/VDDA
- net /MCU/VDDUSB renamed /Block Diagram/Controller/VDDUSB
- net /MCU/VSSA renamed /Block Diagram/Controller/VSSA
- net /MCU/VSS_1 renamed /Block Diagram/Controller/VSS_1
- net /MCU/VSS_2 renamed /Block Diagram/Controller/VSS_2
- net /MCU/VSS_3 renamed /Block Diagram/Controller/VSS_3
- net /Power/+24V0 renamed /Block Diagram/+24V0
- net /Power/0V0 renamed /Block Diagram/M24V0
- net /Power/0V0IN renamed /Block Diagram/Power/0V0IN
- C64 pad 1: /MCU/+5V0 -> /Block Diagram/+5V0
- D2 pad 1: /Power/+5V0_OUT_2 -> /Block Diagram/+5V0
- D2 pad 2: /Power/Buck converter 2/+VOUT -> /Block Diagram/Power/+5V0
- D4 pad 1: /Power/+5V0_OUT_2 -> /Block Diagram/+5V0
- F1 pad 1: /Power/+24V0IN -> /Block Diagram/Power/+24V0IN
- FB3 pad 1: /MCU/+3V3IN -> /Block Diagram/+3V3
- TP1 pad 1: /Power/+5V0_OUT_2 -> /Block Diagram/+5V0
- TP4 pad 1: /Power/+3V3_OUT_3 -> /Block Diagram/+3V3
- U1 pad 1: unconnected-(U1-REGCAPD-Pad1) -> /Block Diagram/ADC/REGCAPD
- U1 pad 10: unconnected-(U1-AIN6/IOUT/VBIAS-Pad10) -> Net-(U1-AIN6/IOUT/VBIAS)
- U1 pad 11: unconnected-(U1-AIN7/IOUT/VBIAS-Pad11) -> Net-(U1-AIN7/IOUT/VBIAS)
- U1 pad 12: unconnected-(U1-REFIN1(+)-Pad12) -> /Block Diagram/ADC/RTD1_REF+
- U1 pad 13: unconnected-(U1-REFIN1(-)-Pad13) -> /Block Diagram/ADC/RTD1_REF-
- U1 pad 14: unconnected-(U1-AIN8/IOUT/VBIAS-Pad14) -> Net-(U1-AIN8/IOUT/VBIAS)
- U1 pad 15: unconnected-(U1-AIN9/IOUT/VBIAS-Pad15) -> Net-(U1-AIN9/IOUT/VBIAS)
- U1 pad 16: unconnected-(U1-AIN10/IOUT/VBIAS-Pad16) -> Net-(U1-AIN10/IOUT/VBIAS)
- U1 pad 17: unconnected-(U1-AIN11/IOUT/VBIAS-Pad17) -> Net-(U1-AIN11/IOUT/VBIAS)
- U1 pad 18: unconnected-(U1-AIN12/IOUT/VBIAS-Pad18) -> Net-(U1-AIN12/IOUT/VBIAS)
- U1 pad 19: unconnected-(U1-AIN13/IOUT/VBIAS-Pad19) -> Net-(U1-AIN13/IOUT/VBIAS)
- U1 pad 2: unconnected-(U1-IOVDD-Pad2) -> /Block Diagram/ADC/IOVDD
- U1 pad 20: unconnected-(U1-AIN14/IOUT/VBIAS/REFIN2(+)-Pad20) -> /Block Diagram/ADC/RTD2_REF+
- U1 pad 21: unconnected-(U1-AIN15/IOUT/VBIAS/REFIN2(-)-Pad21) -> /Block Diagram/ADC/RTD1_REF-
- U1 pad 22: unconnected-(U1-REFOUT-Pad22) -> /Block Diagram/ADC/REFOUT
- U1 pad 23: unconnected-(U1-AVSS-Pad23) -> /Block Diagram/ADC/AVSS
- U1 pad 24: unconnected-(U1-REGCAPA-Pad24) -> /Block Diagram/ADC/REGCAPA
- U1 pad 25: unconnected-(U1-PSW-Pad25) -> /Block Diagram/ADC/RTD1_REF-
- U1 pad 26: unconnected-(U1-AVDD-Pad26) -> /Block Diagram/ADC/AVDD
- U1 pad 27: unconnected-(U1-~{SYNC}-Pad27) -> /Block Diagram/Controller/~{ADC_SYNC}
- U1 pad 28: unconnected-(U1-DOUT/~{RDY}-Pad28) -> /Block Diagram/Controller/SDO/~{IRQ}
- U1 pad 29: unconnected-(U1-DIN-Pad29) -> /Block Diagram/Controller/SDI
- U1 pad 3: unconnected-(U1-DGND-Pad3) -> /Block Diagram/ADC/DGND
- U1 pad 30: unconnected-(U1-SCLK-Pad30) -> /Block Diagram/Controller/SCK
- U1 pad 31: unconnected-(U1-CLK-Pad31) -> /Block Diagram/Controller/ADC_CLK
- U1 pad 32: unconnected-(U1-~{CS}-Pad32) -> /Block Diagram/Controller/~{ADC_CS}
- U1 pad 33: unconnected-(U1-EP-Pad33) -> /Block Diagram/ADC/EP
- U1 pad 4: unconnected-(U1-AIN0/IOUT/VBIAS-Pad4) -> /Block Diagram/ADC/A0+
- U1 pad 5: unconnected-(U1-AIN1/IOUT/VBIAS-Pad5) -> /Block Diagram/ADC/A0-
- U1 pad 6: unconnected-(U1-AIN2/IOUT/VBIAS/P1-Pad6) -> /Block Diagram/ADC/A1+
- U1 pad 7: unconnected-(U1-AIN3/IOUT/VBIAS/P2-Pad7) -> /Block Diagram/ADC/A1-
- U1 pad 8: unconnected-(U1-AIN4/IOUT/VBIAS/P3-Pad8) -> Net-(U1-AIN4/IOUT/VBIAS/P3)
- U1 pad 9: unconnected-(U1-AIN5/IOUT/VBIAS/P4-Pad9) -> Net-(U1-AIN5/IOUT/VBIAS/P4)
- U10 pad 1: /MCU/USB_D+ -> /Block Diagram/Communication/+3V3V
- U10 pad 2: /MCU/USB_D- -> /Block Diagram/Communication/LED2
- U10 pad 3: GND -> /Block Diagram/Communication/LED1
- U10 pad 4: GND -> Net-(U10-XTAL2)
- U10 pad 5: /USB/D- -> Net-(U10-XTAL1/CLKIN)
- U10 pad 6: /USB/D+ -> Net-(U10-VDDCR)
- U2 pad 32: /MCU/USB_D- -> /Block Diagram/Communication/USB_D-
- U2 pad 33: /MCU/USB_D+ -> /Block Diagram/Communication/USB_D+
- U3 pad 1: unconnected-(U3-VCC1-Pad1) -> /Block Diagram/+3V3
- U3 pad 2: unconnected-(U3-IN+-Pad2) -> Net-(U3-IN+)
- U3 pad 3: unconnected-(U3-IN--Pad3) -> GND
- U3 pad 4: unconnected-(U3-GND1-Pad4) -> GND
- U3 pad 5: unconnected-(U3-VCC2-Pad5) -> /Block Diagram/Heater Drive/M15V0
- U3 pad 6: unconnected-(U3-OUTH-Pad6) -> Net-(U3-OUTH)
- U3 pad 7: unconnected-(U3-OUTL-Pad7) -> Net-(U3-OUTL)
- U3 pad 8: unconnected-(U3-VEE2-Pad8) -> /Block Diagram/Heater Drive/+15V0
- U4 pad 1: /Power/+5V0_OUT_2 -> /Block Diagram/+5V0
- U4 pad 2: /Power/+3V3_OUT_3 -> /Block Diagram/+3V3
- U4 pad 3: /Power/Buck converter 2/MOUT -> GND
Routing:
- net GND: track 27.4 -> 0.00 mm
Other:
- board size 80 x 40 mm -> 90 x 75 mm

Commit message: sch improved
Parts:
- removed C29, C32, C33, C34: 1u, Capacitor_SMD:C_0603_1608Metric
- removed C64, C67: 100n, Capacitor_SMD:C_0603_1608Metric
- removed C68: 10u, Capacitor_SMD:C_0805_2012Metric
- removed U7, U8: LP5907MFX-3.3_NOPB, SamacSys_Parts:SOT95P280X145-5N
- added C39: 10u, Capacitor_SMD:C_0805_2012Metric, F.Cu at (160.2, 139.4)
- added C40: 100n, Capacitor_SMD:C_0603_1608Metric, F.Cu at (157.9, 139.6)
- added C41: 4.7u, Capacitor_SMD:C_0805_2012Metric, F.Cu at (158.9, 130.2)
- added C42: 100n, Capacitor_SMD:C_0603_1608Metric, F.Cu at (158.7, 132.6)
- added C43: 100n, Capacitor_SMD:C_0603_1608Metric, F.Cu at (175.0, 56.9)
- added C44: 100n, Capacitor_SMD:C_0603_1608Metric, F.Cu at (175.0, 59.4)
- added C45: 100n, Capacitor_SMD:C_0603_1608Metric, F.Cu at (175.0, 61.9)
- added C46: 100n, Capacitor_SMD:C_0603_1608Metric, F.Cu at (175.0, 64.4)
- added C47: 100n, Capacitor_SMD:C_0603_1608Metric, F.Cu at (175.0, 66.9)
- added C48: 100n, Capacitor_SMD:C_0603_1608Metric, F.Cu at (175.0, 69.4)
- added C49: 100n, Capacitor_SMD:C_0603_1608Metric, F.Cu at (179.0, 56.9)
- added C50: 100n, Capacitor_SMD:C_0603_1608Metric, F.Cu at (179.0, 59.4)
- added C51: 1u, Capacitor_SMD:C_0603_1608Metric, F.Cu at (179.0, 61.9)
- added C52: 1u, Capacitor_SMD:C_0603_1608Metric, F.Cu at (179.0, 64.4)
- added C53: 100n, Capacitor_SMD:C_0603_1608Metric, F.Cu at (179.0, 66.9)
- added C54: 1u, Capacitor_SMD:C_0603_1608Metric, F.Cu at (179.0, 69.4)
- added C55: 100n, Capacitor_SMD:C_0603_1608Metric, F.Cu at (183.0, 56.9)
- added C56: 2.2u, Capacitor_SMD:C_0603_1608Metric, F.Cu at (183.0, 59.4)
- added C57: 2.2u, Capacitor_SMD:C_0603_1608Metric, F.Cu at (183.0, 61.9)
- added PS3: BxxxxS-2WR3, footprints:BxxxxS-2WR3, F.Cu at (129.4, 108.5)
- added PS4: BxxxxS-2WR3, footprints:BxxxxS-2WR3, F.Cu at (102.8, 83.4)
- added U11: STM32H753ZITx, Package_QFP:LQFP-144_20x20mm_P0.5mm, F.Cu at (147.7, 77.1)
- C14: value 100n -> 4.7u
- PS1: value B2415S-1WR3 -> BxxxxS-1WR3; footprint SamacSys_Parts:HLKB2405S2WR3 -> footprints:BxxxxS-1WR3
- PS2: value B2405S-1WR3 -> BxxxxS-1WR3; footprint SamacSys_Parts:HLKB2405S2WR3 -> footprints:BxxxxS-1WR3
- R41, R42, R43, R44, R45, R46, R47, R48, R49, R50, R51, R52, R53, R54, R55, R56: footprint Resistor_SMD:R_0603_1608Metric -> Resistor_SMD:R_0805_2012Metric
- U10: footprint Package_DFN_QFN:VQFN-24-1EP_4x4mm_P0.5mm_EP2.5x2.5mm_ThermalVias -> footprints:VQFN-24-1EP_4x4mm_P0.5mm_EP2.5x2.5mm_ThermalVias
- moved PS2 146.8 mm to (112.8, 88.4)
- moved PS1 127.7 mm to (131.3, 118.9)
- moved SW1 127.2 mm to (119.0, 53.5)
- moved C4 124.0 mm to (106.9, 98.6), turned to 90 degrees
- moved C3 121.8 mm to (109.9, 98.6), turned to 90 degrees
- moved H2 121.5 mm to (105.0, 120.0)
- moved J1 120.8 mm to (103.4, 111.5), turned to -90 degrees
- moved C1 118.7 mm to (102.8, 91.6)
- moved SW2 116.8 mm to (129.6, 53.5)
- moved TP4 116.5 mm to (111.8, 54.9), turned to -90 degrees
- moved Z1 116.3 mm to (114.1, 95.6)
- moved GD1 113.3 mm to (116.8, 110.7), turned to -90 degrees
- moved R1 112.0 mm to (118.0, 96.0)
- moved R59 111.2 mm to (222.5, 71.3)
- moved R60 111.2 mm to (222.5, 73.8)
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Connections:
- C14 pad 1: /Block Diagram/Controller/+3V3V -> /Block Diagram/Controller/MCU Power/VBAT
- C14 pad 2: GND -> GNDD
- C15 pad 1: /Block Diagram/Controller/+3V3V -> /Block Diagram/Controller/MCU Power/VBAT
- C15 pad 2: GND -> GNDD
- C16 pad 2: GND -> /Block Diagram/Controller/VSS
- C17 pad 2: GND -> /Block Diagram/Controller/VSS
- J2 pad 2: /Block Diagram/Interface/RTD1_A -> /Block Diagram/ADC/A0+
- J3 pad 2: /Block Diagram/Interface/RTD2_A -> /Block Diagram/ADC/A1+
- J5 pad 1: /Block Diagram/Heater Drive/+15V0 -> /Block Diagram/Heater Drive/SW_D
- J5 pad 2: /Block Diagram/Heater Drive/SW_G -> /Block Diagram/Heater Drive/+15V0
- J5 pad 3: /Block Diagram/Heater Drive/SW_D -> /Block Diagram/Heater Drive/SW_G
- J8 pad 3: /Block Diagram/Controller/+3V3V -> /Block Diagram/Controller/VDD
- R35 pad 1: /Block Diagram/Controller/+3V3V -> /Block Diagram/Controller/VDD
- R36 pad 2: GND -> /Block Diagram/Controller/VSS
- R38 pad 1: /Block Diagram/Controller/+3V3V -> /Block Diagram/Controller/VDD
- R42 pad 2: /Block Diagram/Interface/RTD1_A -> /Block Diagram/ADC/A0+
- R43 pad 1: Net-(R43-Pad1) -> /Block Diagram/ADC/A0-
- R44 pad 2: Net-(R43-Pad1) -> /Block Diagram/ADC/A0-
- R45 pad 1: /Block Diagram/Interface/+3V3_1 -> /Block Diagram/Interface/+3V3
- R46 pad 2: GND -> /Block Diagram/Interface/0V0
- R51 pad 2: /Block Diagram/Interface/RTD2_A -> /Block Diagram/ADC/A1+
- R52 pad 1: /Block Diagram/Interface/+3V3_2 -> /Block Diagram/Interface/+3V3
- R54 pad 2: GND -> /Block Diagram/Interface/0V0
- R55 pad 2: Net-(R55-Pad2) -> /Block Diagram/ADC/A1-
- R56 pad 1: Net-(R55-Pad2) -> /Block Diagram/ADC/A1-
- SW2 pad 2: GND -> /Block Diagram/Controller/VSS
- U1 pad 2: /Block Diagram/ADC/IOVDD -> /Block Diagram/ADC/D+3V3V
- U1 pad 3: /Block Diagram/ADC/DGND -> GND
- U1 pad 33: /Block Diagram/ADC/EP -> GND
- U2 pad 24: /Block Diagram/Controller/+3V3V -> /Block Diagram/Controller/VDD_1
- U2 pad 48: /Block Diagram/Controller/+3V3V -> /Block Diagram/Controller/VDD_2
Routing:
- net Net-(U3-OUTH): track 0.00 -> 5.06 mm
- net Net-(Q1-G): track 0.00 -> 4.86 mm
- net Net-(U3-OUTL): track 0.00 -> 4.72 mm
- net Net-(U3-IN+): track 0.00 -> 2.79 mm
- net /Block Diagram/Controller/PWMOUT: track 0.00 -> 0.90 mm, vias 0 -> 1
- net GND: vias 0 -> 14
- net /Block Diagram/Power/0V0IN: vias 0 -> 21
- net /Block Diagram/Heater Drive/M15V0: vias 0 -> 5
- net /Block Diagram/+3V3: vias 0 -> 1
- added copper zone on F.Cu, net /Block Diagram/+3V3
- added copper zone on F.Cu, net /Block Diagram/Heater Drive/M15V0
- added copper zone on B.Cu, net /Block Diagram/M24V0
- added copper zone on F.Cu, net /Block Diagram/M24V0
- added copper zone on F.Cu, net /Block Diagram/Power/+24V0IN
- added copper zone on F.Cu, net /Block Diagram/Power/0V0IN
- added copper zone on In1.Cu, net /Block Diagram/Power/0V0IN
- added copper zone on F.Cu, net Earth
- added copper zone on F.Cu, net GND
- added copper zone on In1.Cu, net GND
- added copper zone on F.Cu, net Net-(D11-Pad1)
- added copper zone on F.Cu, net Net-(Q1-D)
Other:
- board size 90 x 75 mm -> 100 x 86.3 mm
- board text added: "All dimensions are in mm unless othjerwise specified."
- board text added: "HEATER"
- board text added: "PWR I/P"
- board text added: "RTD 1"
- board text added: "RTD 2"

Commit message: sch improved
Parts:
- removed C66, C69: 100n, Capacitor_SMD:C_0603_1608Metric
- removed J7: 10118194-0001LF, footprints:101181940001LF
- removed TP3: TestPoint, footprints:TestPoint_THTPad_D1.3mm_Drill0.8mm
- removed U9: USBLC6-4SC6, Package_TO_SOT_SMD:SOT-23-6
- added C10: 10u, Capacitor_SMD:C_0805_2012Metric, F.Cu at (183.0, 56.2)
- added C20: 1u, Capacitor_SMD:C_0603_1608Metric, F.Cu at (175.7, 91.5)
- added C21: 100n, Capacitor_SMD:C_0603_1608Metric, F.Cu at (175.7, 93.6)
- added C29: 100n, Capacitor_SMD:C_0603_1608Metric, F.Cu at (172.1, 96.1)
- added C32: 100n, Capacitor_SMD:C_0603_1608Metric, F.Cu at (165.1, 86.8)
- added C5: 10n, Capacitor_SMD:C_1206_3216Metric, F.Cu at (118.2, 104.7)
- added C58: 1u, Capacitor_SMD:C_0603_1608Metric, F.Cu at (130.2, 117.1)
- added C6: 1u, Capacitor_SMD:C_0805_2012Metric, F.Cu at (124.4, 91.7)
- added C7: 10u, Capacitor_SMD:C_0805_2012Metric, F.Cu at (102.7, 84.0)
- added C8: 10u, Capacitor_SMD:C_0805_2012Metric, F.Cu at (115.2, 85.8)
- added C9: 100n, Capacitor_SMD:C_0603_1608Metric, F.Cu at (175.6, 103.5)
- added D1: PESD3V3S1UL, Diode_SMD:D_SOD-882, F.Cu at (112.2, 73.4)
- added D5: ESD9X5.0ST5G, SamacSys_Parts:SODFL1006X40N, F.Cu at (189.9, 61.3)
- added J9: USB4930-00-A, footprints:USB4930-00-A, F.Cu at (196.3, 65.4)
- added R86: 10k, Resistor_SMD:R_0603_1608Metric, F.Cu at (125.8, 57.4)
- added R87: 10k, Resistor_SMD:R_0603_1608Metric, F.Cu at (163.2, 75.4)
- added R88: 0R, Resistor_SMD:R_0805_2012Metric, F.Cu at (180.1, 110.0)
- added R89: 0R, Resistor_SMD:R_0805_2012Metric, F.Cu at (180.1, 107.0)
- added R90: 5.1k, Resistor_SMD:R_0603_1608Metric, F.Cu at (182.8, 61.5)
- added R91: 100R, Resistor_SMD:R_0603_1608Metric, F.Cu at (125.8, 53.2)
- C12: value 10u -> 100n; footprint Capacitor_SMD:C_0805_2012Metric -> Capacitor_SMD:C_0603_1608Metric
- C14, C15, C19, C22, C23, C26, C30, C43, C44, C45, C46, C47, C48, C49, C50, C51, C52, C53, C54, C55, C56, C57, R57, R58, R59, R60, R61, R64, R69, R70, R71, R72: moved to B.Cu
- C18: value 100n -> 1u
- C27: value 1u -> 100n
- C31, C38: value 100n -> 22n; moved to B.Cu
- R37: value 1k2 -> 6R2
- R39: value 1k2 -> 10R
- R68: value 0R -> 10k
- R76: value 4k7 -> 5.1k
- TP2: value TestPoint -> 24V RAW; footprint footprints:TestPoint_THTPad_D1.3mm_Drill0.8mm -> Connector_PinSocket_2.54mm:PinSocket_1x02_P2.54mm_Vertical
- U2: value STM32L412CxTx -> NUP4106DR2G; footprint SamacSys_Parts:QFP50P900X900X160-48N -> SamacSys_Parts:SOIC127P600X175-8N
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Connections:
- C11 pad 1: /Block Diagram/Controller/+3V3V -> /Block Diagram/Controller/VDD
- C11 pad 2: GND -> GNDD
- C12 pad 1: /Block Diagram/ADC/D+3V3V -> /Block Diagram/+5V0
- C12 pad 2: GND -> GNDD
- C13 pad 2: GND -> GNDD
- C14 pad 1: /Block Diagram/Controller/MCU Power/VBAT -> /Block Diagram/Controller/VDD
- C15 pad 1: /Block Diagram/Controller/MCU Power/VBAT -> /Block Diagram/Controller/VDD
- C16 pad 1: /Block Diagram/Controller/BOOT0 -> /Block Diagram/Controller/MCU GPIO/BOOT0
- C16 pad 2: /Block Diagram/Controller/VSS -> GNDD
- C17 pad 2: /Block Diagram/Controller/VSS -> GNDD
- C18 pad 1: /Block Diagram/ADC/D+3V3V -> /Block Diagram/+5V0
- C18 pad 2: GND -> GNDD
- C19 pad 2: GND -> GNDD
- C2 pad 1: V_BUS -> GNDD
- C2 pad 2: GND -> V_BUS
- C22 pad 2: GND -> GNDD
- C23 pad 2: GND -> GNDD
- C24 pad 1: GND -> GNDD
- C24 pad 2: Net-(C24-Pad2) -> Net-(U10-XTAL1/CLKIN)
- C25 pad 1: GND -> GNDD
- C26 pad 2: GND -> GNDD
- C27 pad 1: /Block Diagram/+5V0 -> /Block Diagram/ADC/REGCAPD
- C27 pad 2: GND -> GNDD
- C28 pad 2: GND -> GNDD
- C30 pad 2: GND -> GNDD
- C31 pad 1: Net-(J6-RCT) -> /Block Diagram/Communication/+3V3V
- C31 pad 2: GND -> GNDD
- C38 pad 1: Net-(J6-RCT) -> /Block Diagram/Communication/+3V3V
- C38 pad 2: GND -> GNDD
- C41 pad 2: GND -> GNDD
- C42 pad 2: GND -> GNDD
- C43 pad 1: /Block Diagram/Controller/MCU Power/VBAT -> /Block Diagram/Controller/VDD
- C44 pad 1: /Block Diagram/Controller/MCU Power/VBAT -> /Block Diagram/Controller/VDD
- C45 pad 1: /Block Diagram/Controller/MCU Power/VBAT -> /Block Diagram/Controller/VDD
- C46 pad 1: /Block Diagram/Controller/MCU Power/VBAT -> /Block Diagram/Controller/VDD
- C47 pad 1: /Block Diagram/Controller/MCU Power/VBAT -> /Block Diagram/Controller/VDD
- C48 pad 1: /Block Diagram/Controller/MCU Power/VBAT -> /Block Diagram/Controller/VDD
- C49 pad 1: /Block Diagram/Controller/MCU Power/VBAT -> /Block Diagram/Controller/VDD
- C50 pad 1: /Block Diagram/Controller/MCU Power/VBAT -> /Block Diagram/Controller/VDD
- C51 pad 1: /Block Diagram/Controller/MCU Power/VBAT -> /Block Diagram/Controller/VDD
- C52 pad 1: /Block Diagram/Controller/MCU Power/VBAT -> /Block Diagram/Controller/VDD
- C53 pad 1: /Block Diagram/Controller/MCU Power/VBAT -> /Block Diagram/Controller/VDD
- C54 pad 1: /Block Diagram/Controller/MCU Power/VBAT -> /Block Diagram/Controller/VDD
- C55 pad 1: /Block Diagram/Controller/MCU Power/VBAT -> /Block Diagram/Controller/VDD
- FB3 pad 2: /Block Diagram/Controller/+3V3V -> /Block Diagram/Controller/VDD
- FB7 pad 1: GND -> GNDD
- FB8 pad 1: /Block Diagram/Communication/VCC_USB -> /Block Diagram/Communication/USB_VBUS
- J5 pad 2: /Block Diagram/Heater Drive/+15V0 -> /Block Diagram/Heater Drive/M15V0
- J6 pad 3: /Block Diagram/Communication/PD_P -> /Block Diagram/Communication/RD_P
- J6 pad 4: Net-(J6-RCT) -> /Block Diagram/Communication/+3V3V
- J6 pad 5: Net-(J6-RCT) -> /Block Diagram/Communication/+3V3V
- J6 pad 8: Net-(C35-Pad1) -> GND_SHIELD
- J6 pad SH: GND_SHIELD -> Net-(C35-Pad1)
- J8 pad 11: GND -> /Block Diagram/Controller/GNDDETECT
- J8 pad 5: GND -> GNDD
- J8 pad 7: GND -> GNDD
- PS2 pad 3: GND -> GNDD
- PS4 pad 4: GND -> GNDD
- R27 pad 2: /Block Diagram/Heater Drive/+15V0 -> /Block Diagram/Heater Drive/M15V0
- R36 pad 1: /Block Diagram/Controller/BOOT0 -> /Block Diagram/Controller/MCU GPIO/BOOT0
- R36 pad 2: /Block Diagram/Controller/VSS -> GNDD
- R38 pad 2: /Block Diagram/Controller/NRST -> /Block Diagram/Controller/MCU GPIO/PDR_ON
- R40 pad 1: /Block Diagram/Controller/PWMOUT -> /Block Diagram/Controller/MCU GPIO/PE9
- R45 pad 1: /Block Diagram/Interface/+3V3 -> /Block Diagram/ADC/A+3V3
- R46 pad 2: /Block Diagram/Interface/0V0 -> GNDD
- R52 pad 1: /Block Diagram/Interface/+3V3 -> /Block Diagram/ADC/A+3V3
- R54 pad 2: /Block Diagram/Interface/0V0 -> GNDD
- R60 pad 2: /Block Diagram/Communication/RMII_MDIO -> /Block Diagram/Controller/MCU GPIO/PA2
- R62 pad 1: /Block Diagram/Communication/RMII_RXD0 -> /Block Diagram/Controller/MCU GPIO/PC4
- R63 pad 1: /Block Diagram/Communication/RMII_RXD1 -> /Block Diagram/Controller/MCU GPIO/PC5
- R64 pad 1: GND -> GNDD
- R65 pad 1: /Block Diagram/Communication/RMII_CRS_DV -> /Block Diagram/Controller/MCU GPIO/PA7
- R66 pad 1: /Block Diagram/Communication/RMII_REF_CLK -> /Block Diagram/Controller/MCU GPIO/PA1
- R68 pad 1: Net-(C24-Pad2) -> /Block Diagram/Communication/USB_VBUS
- R68 pad 2: Net-(U10-XTAL1/CLKIN) -> /Block Diagram/Controller/MCU GPIO/PA9
- R71 pad 2: /Block Diagram/Communication/PD_P -> /Block Diagram/Communication/RD_P
- R73 pad 2: GND -> GNDD
- R74 pad 2: GND -> GNDD
- R75 pad 2: GND -> GNDD
- R76 pad 1: Net-(U1-AIN4/IOUT/VBIAS/P3) -> Net-(J9-CC1)
- R76 pad 2: /Block Diagram/ADC/AVSS -> GNDD
- R77 pad 2: /Block Diagram/ADC/AVSS -> GNDD
- R78 pad 2: /Block Diagram/ADC/AVSS -> GNDD
- R79 pad 2: /Block Diagram/ADC/AVSS -> GNDD
- R80 pad 2: /Block Diagram/ADC/AVSS -> GNDD
- R81 pad 2: /Block Diagram/ADC/AVSS -> GNDD
- R82 pad 2: /Block Diagram/ADC/AVSS -> GNDD
- R83 pad 2: /Block Diagram/ADC/AVSS -> GNDD
- R84 pad 2: /Block Diagram/ADC/AVSS -> GNDD
- R85 pad 2: /Block Diagram/ADC/AVSS -> GNDD
- SW1 pad 1: Net-(R35-Pad2) -> /Block Diagram/Controller/MCU GPIO/BOOT0
- SW1 pad 2: /Block Diagram/Controller/BOOT0 -> Net-(R35-Pad2)
- SW2 pad 2: /Block Diagram/Controller/VSS -> GNDD
- U1 pad 22: /Block Diagram/ADC/REFOUT -> /Block Diagram/ADC/REFVOUT
- U1 pad 23: /Block Diagram/ADC/AVSS -> GNDD
- U1 pad 26: /Block Diagram/ADC/AVDD -> /Block Diagram/ADC/A+3V3
- U1 pad 27: /Block Diagram/Controller/~{ADC_SYNC} -> /Block Diagram/Controller/MCU GPIO/PE15
- U1 pad 28: /Block Diagram/Controller/SDO/~{IRQ} -> /Block Diagram/Controller/MCU GPIO/PB14
- U1 pad 29: /Block Diagram/Controller/SDI -> /Block Diagram/Controller/MCU GPIO/PB15
- U1 pad 3: GND -> GNDD
- U1 pad 30: /Block Diagram/Controller/SCK -> /Block Diagram/Controller/MCU GPIO/PB10
- U1 pad 31: /Block Diagram/Controller/ADC_CLK -> /Block Diagram/Controller/MCU GPIO/PA8
- U1 pad 32: /Block Diagram/Controller/~{ADC_CS} -> /Block Diagram/Controller/MCU GPIO/PD11
- U1 pad 33: GND -> GNDD
- U1 pad 8: Net-(U1-AIN4/IOUT/VBIAS/P3) -> /Block Diagram/ADC/REFIOUT
- U10 pad 12: /Block Diagram/Communication/RMII_MDIO -> /Block Diagram/Controller/MCU GPIO/PA2
- U10 pad 13: /Block Diagram/Communication/RMII_MDC -> /Block Diagram/Controller/MCU GPIO/PC1
- U10 pad 16: /Block Diagram/Communication/RMII_TX_EN -> /Block Diagram/Controller/MCU GPIO/PG11
- U10 pad 17: /Block Diagram/Communication/RMII_TXD0 -> /Block Diagram/Controller/MCU GPIO/PG13
- U10 pad 18: /Block Diagram/Communication/RMII_TXD1 -> /Block Diagram/Controller/MCU GPIO/PB13
- U10 pad 20: /Block Diagram/Communication/TD_N -> /Block Diagram/Communication/TD_P
- U10 pad 21: /Block Diagram/Communication/TD_P -> /Block Diagram/Communication/TD_N
- U10 pad 22: /Block Diagram/Communication/RD_N -> /Block Diagram/Communication/RD_P
- U10 pad 23: /Block Diagram/Communication/PD_P -> /Block Diagram/Communication/RD_N
- U10 pad 25: GND -> GNDD
- U11 pad 1: unconnected-(U11B-PE2-Pad1) -> /Block Diagram/Controller/MCU GPIO/PE2
- U11 pad 10: unconnected-(U11B-PF0-Pad10) -> /Block Diagram/Controller/MCU GPIO/PF0
- U11 pad 100: unconnected-(U11A-PA8-Pad100) -> /Block Diagram/Controller/MCU GPIO/PA8
- U11 pad 101: unconnected-(U11A-PA9-Pad101) -> /Block Diagram/Controller/MCU GPIO/PA9
- U11 pad 102: unconnected-(U11A-PA10-Pad102) -> /Block Diagram/Controller/MCU GPIO/PA10
- U11 pad 103: unconnected-(U11A-PA11-Pad103) -> /Block Diagram/Communication/USB_D+
- U11 pad 104: unconnected-(U11A-PA12-Pad104) -> /Block Diagram/Communication/USB_D-
- U11 pad 105: unconnected-(U11A-PA13-Pad105) -> /Block Diagram/Controller/SWDIO
- U11 pad 108: /Block Diagram/Controller/MCU Power/VBAT -> /Block Diagram/Controller/VDD
- U11 pad 109: unconnected-(U11A-PA14-Pad109) -> /Block Diagram/Controller/SWCLK
- U11 pad 11: unconnected-(U11B-PF1-Pad11) -> /Block Diagram/Controller/MCU GPIO/PF1
- U11 pad 110: unconnected-(U11A-PA15-Pad110) -> /Block Diagram/Controller/MCU GPIO/PA15
- U11 pad 111: unconnected-(U11A-PC10-Pad111) -> /Block Diagram/Controller/LOG_TX
- U11 pad 112: unconnected-(U11A-PC11-Pad112) -> /Block Diagram/Controller/LOG_RX
- U11 pad 113: unconnected-(U11A-PC12-Pad113) -> /Block Diagram/Controller/MCU GPIO/PC12
- U11 pad 114: unconnected-(U11B-PD0-Pad114) -> /Block Diagram/Controller/MCU GPIO/PD0
- U11 pad 115: unconnected-(U11B-PD1-Pad115) -> /Block Diagram/Controller/MCU GPIO/PD1
- U11 pad 116: unconnected-(U11B-PD2-Pad116) -> /Block Diagram/Controller/MCU GPIO/PD2
- U11 pad 117: unconnected-(U11B-PD3-Pad117) -> /Block Diagram/Controller/MCU GPIO/PD3
- U11 pad 118: unconnected-(U11B-PD4-Pad118) -> /Block Diagram/Controller/MCU GPIO/PD4
- U11 pad 119: unconnected-(U11B-PD5-Pad119) -> /Block Diagram/Controller/MCU GPIO/PD5
- U11 pad 12: unconnected-(U11B-PF2-Pad12) -> /Block Diagram/Controller/MCU GPIO/PF2
- U11 pad 121: /Block Diagram/Controller/MCU Power/VBAT -> /Block Diagram/Controller/VDD
- U11 pad 122: unconnected-(U11B-PD6-Pad122) -> /Block Diagram/Controller/MCU GPIO/PD6
- U11 pad 123: unconnected-(U11B-PD7-Pad123) -> /Block Diagram/Controller/MCU GPIO/PD7
- U11 pad 124: unconnected-(U11B-PG9-Pad124) -> /Block Diagram/Controller/MCU GPIO/PG9
- U11 pad 125: unconnected-(U11B-PG10-Pad125) -> /Block Diagram/Controller/MCU GPIO/PG10
- U11 pad 126: unconnected-(U11B-PG11-Pad126) -> /Block Diagram/Controller/MCU GPIO/PG11
- U11 pad 127: unconnected-(U11B-PG12-Pad127) -> /Block Diagram/Controller/MCU GPIO/PG12
- U11 pad 128: unconnected-(U11B-PG13-Pad128) -> /Block Diagram/Controller/MCU GPIO/PG13
- U11 pad 129: unconnected-(U11B-PG14-Pad129) -> /Block Diagram/Controller/MCU GPIO/PG14
- U11 pad 13: unconnected-(U11B-PF3-Pad13) -> /Block Diagram/Controller/MCU GPIO/PF3
- U11 pad 131: /Block Diagram/Controller/MCU Power/VBAT -> /Block Diagram/Controller/VDD
- U11 pad 132: unconnected-(U11B-PG15-Pad132) -> /Block Diagram/Controller/MCU GPIO/PG15
- U11 pad 133: unconnected-(U11A-PB3-Pad133) -> /Block Diagram/Controller/SWO
- U11 pad 134: unconnected-(U11A-PB4-Pad134) -> /Block Diagram/Controller/MCU GPIO/PB4
- U11 pad 135: unconnected-(U11A-PB5-Pad135) -> /Block Diagram/Controller/MCU GPIO/PB5
- U11 pad 136: unconnected-(U11A-PB6-Pad136) -> /Block Diagram/Controller/MCU GPIO/PB6
- U11 pad 137: unconnected-(U11A-PB7-Pad137) -> /Block Diagram/Controller/MCU GPIO/PB7
- U11 pad 138: unconnected-(U11A-BOOT0-Pad138) -> /Block Diagram/Controller/MCU GPIO/BOOT0
- U11 pad 139: unconnected-(U11A-PB8-Pad139) -> /Block Diagram/Controller/MCU GPIO/PB8
- U11 pad 14: unconnected-(U11B-PF4-Pad14) -> /Block Diagram/Controller/MCU GPIO/PF4
- U11 pad 140: unconnected-(U11A-PB9-Pad140) -> /Block Diagram/Controller/MCU GPIO/PB9
- U11 pad 141: unconnected-(U11B-PE0-Pad141) -> /Block Diagram/Controller/MCU GPIO/PE0
- U11 pad 142: unconnected-(U11B-PE1-Pad142) -> /Block Diagram/Controller/MCU GPIO/PE1
- U11 pad 143: unconnected-(U11A-PDR_ON-Pad143) -> /Block Diagram/Controller/MCU GPIO/PDR_ON
- U11 pad 144: /Block Diagram/Controller/MCU Power/VBAT -> /Block Diagram/Controller/VDD
- U11 pad 15: unconnected-(U11B-PF5-Pad15) -> /Block Diagram/Controller/MCU GPIO/PF5
- U11 pad 17: /Block Diagram/Controller/MCU Power/VBAT -> /Block Diagram/Controller/VDD
- U11 pad 18: unconnected-(U11B-PF6-Pad18) -> /Block Diagram/Controller/MCU GPIO/PF6
- U11 pad 19: unconnected-(U11B-PF7-Pad19) -> /Block Diagram/Controller/MCU GPIO/PF7
- U11 pad 2: unconnected-(U11B-PE3-Pad2) -> /Block Diagram/Controller/MCU GPIO/PE3
- U11 pad 20: unconnected-(U11B-PF8-Pad20) -> /Block Diagram/Controller/MCU GPIO/PF8
- U11 pad 21: unconnected-(U11B-PF9-Pad21) -> /Block Diagram/Controller/MCU GPIO/PF9
- U11 pad 22: unconnected-(U11B-PF10-Pad22) -> /Block Diagram/Controller/MCU GPIO/PF10
- U11 pad 23: unconnected-(U11A-PH0-Pad23) -> /Block Diagram/Controller/MCU GPIO/RCC_OSC_IN
- U11 pad 24: unconnected-(U11A-PH1-Pad24) -> /Block Diagram/Controller/MCU GPIO/RCC_OSC_OUT
- U11 pad 25: unconnected-(U11A-NRST-Pad25) -> /Block Diagram/Controller/NRST
- U11 pad 26: unconnected-(U11A-PC0-Pad26) -> /Block Diagram/Controller/MCU GPIO/PC0
- U11 pad 27: unconnected-(U11A-PC1-Pad27) -> /Block Diagram/Controller/MCU GPIO/PC1
- U11 pad 28: unconnected-(U11A-PC2_C-Pad28) -> /Block Diagram/Controller/MCU GPIO/PC2
- U11 pad 29: unconnected-(U11A-PC3_C-Pad29) -> /Block Diagram/Controller/MCU GPIO/PC3
- U11 pad 3: unconnected-(U11B-PE4-Pad3) -> /Block Diagram/Controller/MCU GPIO/PE4
- U11 pad 30: /Block Diagram/Controller/MCU Power/VBAT -> /Block Diagram/Controller/VDD
- U11 pad 32: /Block Diagram/Controller/MCU Power/VBAT -> /Block Diagram/Controller/VDD
- U11 pad 33: /Block Diagram/Controller/MCU Power/VBAT -> /Block Diagram/Controller/VDD
- U11 pad 34: unconnected-(U11A-PA0-Pad34) -> /Block Diagram/Controller/MCU GPIO/PA0
- U11 pad 35: unconnected-(U11A-PA1-Pad35) -> /Block Diagram/Controller/MCU GPIO/PA1
- U11 pad 36: unconnected-(U11A-PA2-Pad36) -> /Block Diagram/Controller/MCU GPIO/PA2
- U11 pad 37: unconnected-(U11A-PA3-Pad37) -> /Block Diagram/Controller/MCU GPIO/PA3
- U11 pad 39: /Block Diagram/Controller/MCU Power/VBAT -> /Block Diagram/Controller/VDD
- U11 pad 4: unconnected-(U11B-PE5-Pad4) -> /Block Diagram/Controller/MCU GPIO/PE5
- U11 pad 40: unconnected-(U11A-PA4-Pad40) -> /Block Diagram/Controller/MCU GPIO/PA4
- U11 pad 41: unconnected-(U11A-PA5-Pad41) -> /Block Diagram/Controller/MCU GPIO/PA5
- U11 pad 42: unconnected-(U11A-PA6-Pad42) -> /Block Diagram/Controller/MCU GPIO/PA6
- U11 pad 43: unconnected-(U11A-PA7-Pad43) -> /Block Diagram/Controller/MCU GPIO/PA7
- U11 pad 44: unconnected-(U11A-PC4-Pad44) -> /Block Diagram/Controller/MCU GPIO/PC4
- U11 pad 45: unconnected-(U11A-PC5-Pad45) -> /Block Diagram/Controller/MCU GPIO/PC5
- U11 pad 46: unconnected-(U11A-PB0-Pad46) -> /Block Diagram/Controller/MCU GPIO/PB0
- U11 pad 47: unconnected-(U11A-PB1-Pad47) -> /Block Diagram/Controller/MCU GPIO/PB1
- U11 pad 48: unconnected-(U11A-PB2-Pad48) -> /Block Diagram/Controller/MCU GPIO/PB2
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Routing:
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- added copper zone on F.Cu, net /Block Diagram/+24V0
- added copper zone on F.Cu, net /Block Diagram/Heater Drive/+15V0
- added copper zone on In1.Cu, net /Block Diagram/Heater Drive/M15V0
- added copper zone on In1.Cu, net /Block Diagram/M24V0
- added copper zone on F.Cu, net GNDD
- added copper zone on In1.Cu, net Net-(FB7-Pad2)
- removed copper zone on B.Cu, net /Block Diagram/M24V0
- removed copper zone on F.Cu, net GND
- removed copper zone on In1.Cu, net GND
Other:
- board size 100 x 86.3 mm -> 100 x 75 mm
- board text added: "1"
- board text added: "2"
- board text added: "3"
- board text added: "4"
- board text added: "NSMB-STM32-V1.0.0"
