File: cryonano-nano-stage/cryonano-nano-stage.kicad_pcb (KiCad board)
At the start: 4 copper layers, 100 x 75 mm, 173 parts, among them J1 24VDC IN, J2 JST-B2B-XH-AM, J3 JST-B2B-XH-AM, J5 JST-B3B-XH-AM, J6 RJ45_Hanrun_HR911105A_Horizon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, J8 Conn_ST_STDC14, J9 USB4930-00-A, Q1 PMV100EPAR, SW1 BOOT, SW2 RESET, U1 AD7124-8BCPZ-RL7, U10 LAN8742A, U2 NUP4106DR2G, U3 1ED3141MU12FXUMA1, U4 AP7363-33D-13, U5 ECMF02-2AMX6, U6 LP5907MFX-3.3_NOPB, U7 STM32H753ZITx, Y3 25.0MHz

Commit message: complete
Parts:
- moved TP1 65.8 mm to (103.8, 120.0)
- moved TP2 23.1 mm to (88.0, 87.8)
- moved R93 1.75 mm to (43.2, 93.7), turned to 180 degrees
- moved D4 1.28 mm to (43.3, 96.0), turned to 180 degrees
Connections:
- net /Block Diagram/Controller/MCU GPIO/PA1 renamed /Block Diagram/Communication/RMII_REF_CLK
- net /Block Diagram/Controller/MCU GPIO/PA10 renamed /Block Diagram/Controller/ID
- net /Block Diagram/Controller/MCU GPIO/PA2 renamed /Block Diagram/Communication/RMII_MDIO
- net /Block Diagram/Controller/MCU GPIO/PA7 renamed /Block Diagram/Communication/RMII_CRS_DV
- net /Block Diagram/Controller/MCU GPIO/PA8 renamed Net-(U7A-PA8)
- net /Block Diagram/Controller/MCU GPIO/PA9 renamed Net-(U7A-PA9)
- net /Block Diagram/Controller/MCU GPIO/PB11 renamed /Block Diagram/Communication/RMII_TX_EN
- net /Block Diagram/Controller/MCU GPIO/PB12 renamed /Block Diagram/Communication/RMII_TXD0
- net /Block Diagram/Controller/MCU GPIO/PB13 renamed /Block Diagram/Communication/RMII_TXD1
- net /Block Diagram/Controller/MCU GPIO/PB6 renamed Net-(TP3-Pin_1)
- net /Block Diagram/Controller/MCU GPIO/PB7 renamed Net-(TP3-Pin_2)
- net /Block Diagram/Controller/MCU GPIO/PC1 renamed /Block Diagram/Communication/RMII_MDC
- net /Block Diagram/Controller/MCU GPIO/PC4 renamed /Block Diagram/Communication/RMII_RXD0
- net /Block Diagram/Controller/MCU GPIO/PC5 renamed /Block Diagram/Communication/RMII_RXD1
- net /Block Diagram/Controller/MCU GPIO/PC9 renamed /Block Diagram/ADC/CLK
- net /Block Diagram/Controller/MCU GPIO/PE10 renamed /Block Diagram/ADC/DOUT/~{RDY}
- net /Block Diagram/Controller/MCU GPIO/PE11 renamed /Block Diagram/ADC/~{CS}
- net /Block Diagram/Controller/MCU GPIO/PE12 renamed /Block Diagram/ADC/SCLK
- net /Block Diagram/Controller/MCU GPIO/PE14 renamed /Block Diagram/ADC/DIN
- net /Block Diagram/Controller/MCU GPIO/PE15 renamed /Block Diagram/ADC/~{SYNC}
- net /Block Diagram/Controller/MCU GPIO/PE9 renamed /Block Diagram/Controller/PWMOUT
- U7 pad 1: /Block Diagram/Controller/MCU GPIO/PE2 -> unconnected-(U7B-PE2-Pad1)
- U7 pad 10: /Block Diagram/Controller/MCU GPIO/PF0 -> unconnected-(U7B-PF0-Pad10)
- U7 pad 11: /Block Diagram/Controller/MCU GPIO/PF1 -> unconnected-(U7B-PF1-Pad11)
- U7 pad 110: /Block Diagram/Controller/MCU GPIO/PA15 -> unconnected-(U7A-PA15-Pad110)
- U7 pad 113: /Block Diagram/Controller/MCU GPIO/PC12 -> unconnected-(U7A-PC12-Pad113)
- U7 pad 114: /Block Diagram/Controller/MCU GPIO/PD0 -> unconnected-(U7B-PD0-Pad114)
- U7 pad 115: /Block Diagram/Controller/MCU GPIO/PD1 -> unconnected-(U7B-PD1-Pad115)
- U7 pad 116: /Block Diagram/Controller/MCU GPIO/PD2 -> unconnected-(U7B-PD2-Pad116)
- U7 pad 117: /Block Diagram/Controller/MCU GPIO/PD3 -> unconnected-(U7B-PD3-Pad117)
- U7 pad 118: /Block Diagram/Controller/MCU GPIO/PD4 -> unconnected-(U7B-PD4-Pad118)
- U7 pad 119: /Block Diagram/Controller/MCU GPIO/PD5 -> unconnected-(U7B-PD5-Pad119)
- U7 pad 12: /Block Diagram/Controller/MCU GPIO/PF2 -> unconnected-(U7B-PF2-Pad12)
- U7 pad 122: /Block Diagram/Controller/MCU GPIO/PD6 -> unconnected-(U7B-PD6-Pad122)
- U7 pad 123: /Block Diagram/Controller/MCU GPIO/PD7 -> unconnected-(U7B-PD7-Pad123)
- U7 pad 124: /Block Diagram/Controller/MCU GPIO/PG9 -> unconnected-(U7B-PG9-Pad124)
- U7 pad 125: /Block Diagram/Controller/MCU GPIO/PG10 -> unconnected-(U7B-PG10-Pad125)
- U7 pad 126: /Block Diagram/Controller/MCU GPIO/PG11 -> unconnected-(U7B-PG11-Pad126)
- U7 pad 127: /Block Diagram/Controller/MCU GPIO/PG12 -> unconnected-(U7B-PG12-Pad127)
- U7 pad 128: /Block Diagram/Controller/MCU GPIO/PG13 -> unconnected-(U7B-PG13-Pad128)
- U7 pad 129: /Block Diagram/Controller/MCU GPIO/PG14 -> unconnected-(U7B-PG14-Pad129)
- U7 pad 13: /Block Diagram/Controller/MCU GPIO/PF3 -> unconnected-(U7B-PF3-Pad13)
- U7 pad 132: /Block Diagram/Controller/MCU GPIO/PG15 -> unconnected-(U7B-PG15-Pad132)
- U7 pad 134: /Block Diagram/Controller/MCU GPIO/PB4 -> unconnected-(U7A-PB4-Pad134)
- U7 pad 135: /Block Diagram/Controller/MCU GPIO/PB5 -> unconnected-(U7A-PB5-Pad135)
- U7 pad 139: /Block Diagram/Controller/MCU GPIO/PB8 -> unconnected-(U7A-PB8-Pad139)
- U7 pad 14: /Block Diagram/Controller/MCU GPIO/PF4 -> unconnected-(U7B-PF4-Pad14)
- U7 pad 140: /Block Diagram/Controller/MCU GPIO/PB9 -> unconnected-(U7A-PB9-Pad140)
- U7 pad 141: /Block Diagram/Controller/MCU GPIO/PE0 -> unconnected-(U7B-PE0-Pad141)
- U7 pad 142: /Block Diagram/Controller/MCU GPIO/PE1 -> unconnected-(U7B-PE1-Pad142)
- U7 pad 15: /Block Diagram/Controller/MCU GPIO/PF5 -> unconnected-(U7B-PF5-Pad15)
- U7 pad 18: /Block Diagram/Controller/MCU GPIO/PF6 -> unconnected-(U7B-PF6-Pad18)
- U7 pad 19: /Block Diagram/Controller/MCU GPIO/PF7 -> unconnected-(U7B-PF7-Pad19)
- U7 pad 2: /Block Diagram/Controller/MCU GPIO/PE3 -> unconnected-(U7B-PE3-Pad2)
- U7 pad 20: /Block Diagram/Controller/MCU GPIO/PF8 -> unconnected-(U7B-PF8-Pad20)
- U7 pad 21: /Block Diagram/Controller/MCU GPIO/PF9 -> unconnected-(U7B-PF9-Pad21)
- U7 pad 22: /Block Diagram/Controller/MCU GPIO/PF10 -> unconnected-(U7B-PF10-Pad22)
- U7 pad 26: /Block Diagram/Controller/MCU GPIO/PC0 -> unconnected-(U7A-PC0-Pad26)
- U7 pad 28: /Block Diagram/Controller/MCU GPIO/PC2 -> unconnected-(U7A-PC2_C-Pad28)
- U7 pad 29: /Block Diagram/Controller/MCU GPIO/PC3 -> unconnected-(U7A-PC3_C-Pad29)
- U7 pad 3: /Block Diagram/Controller/MCU GPIO/PE4 -> unconnected-(U7B-PE4-Pad3)
- U7 pad 34: /Block Diagram/Controller/MCU GPIO/PA0 -> unconnected-(U7A-PA0-Pad34)
- U7 pad 37: /Block Diagram/Controller/MCU GPIO/PA3 -> unconnected-(U7A-PA3-Pad37)
- U7 pad 4: /Block Diagram/Controller/MCU GPIO/PE5 -> unconnected-(U7B-PE5-Pad4)
- U7 pad 40: /Block Diagram/Controller/MCU GPIO/PA4 -> unconnected-(U7A-PA4-Pad40)
- U7 pad 41: /Block Diagram/Controller/MCU GPIO/PA5 -> unconnected-(U7A-PA5-Pad41)
- U7 pad 42: /Block Diagram/Controller/MCU GPIO/PA6 -> unconnected-(U7A-PA6-Pad42)
- U7 pad 46: /Block Diagram/Controller/MCU GPIO/PB0 -> unconnected-(U7A-PB0-Pad46)
- U7 pad 47: /Block Diagram/Controller/MCU GPIO/PB1 -> unconnected-(U7A-PB1-Pad47)
- U7 pad 48: /Block Diagram/Controller/MCU GPIO/PB2 -> unconnected-(U7A-PB2-Pad48)
- U7 pad 49: /Block Diagram/Controller/MCU GPIO/PF11 -> unconnected-(U7B-PF11-Pad49)
- U7 pad 5: /Block Diagram/Controller/MCU GPIO/PE6 -> unconnected-(U7B-PE6-Pad5)
- U7 pad 50: /Block Diagram/Controller/MCU GPIO/PF12 -> unconnected-(U7B-PF12-Pad50)
- U7 pad 53: /Block Diagram/Controller/MCU GPIO/PF13 -> unconnected-(U7B-PF13-Pad53)
- U7 pad 54: /Block Diagram/Controller/MCU GPIO/PF14 -> unconnected-(U7B-PF14-Pad54)
- U7 pad 55: /Block Diagram/Controller/MCU GPIO/PF15 -> unconnected-(U7B-PF15-Pad55)
- U7 pad 56: /Block Diagram/Controller/MCU GPIO/PG0 -> unconnected-(U7B-PG0-Pad56)
- U7 pad 57: /Block Diagram/Controller/MCU GPIO/PG1 -> unconnected-(U7B-PG1-Pad57)
- U7 pad 58: /Block Diagram/Controller/MCU GPIO/PE7 -> unconnected-(U7B-PE7-Pad58)
- U7 pad 59: /Block Diagram/Controller/MCU GPIO/PE8 -> unconnected-(U7B-PE8-Pad59)
- U7 pad 69: /Block Diagram/Controller/MCU GPIO/PB10 -> unconnected-(U7A-PB10-Pad69)
- U7 pad 7: /Block Diagram/Controller/MCU GPIO/PC13 -> unconnected-(U7A-PC13-Pad7)
- U7 pad 75: /Block Diagram/Controller/MCU GPIO/PB14 -> unconnected-(U7A-PB14-Pad75)
- U7 pad 76: /Block Diagram/Controller/MCU GPIO/PB15 -> unconnected-(U7A-PB15-Pad76)
- U7 pad 77: /Block Diagram/Controller/MCU GPIO/PD8 -> unconnected-(U7B-PD8-Pad77)
- U7 pad 78: /Block Diagram/Controller/MCU GPIO/PD9 -> unconnected-(U7B-PD9-Pad78)
- U7 pad 79: /Block Diagram/Controller/MCU GPIO/PD10 -> unconnected-(U7B-PD10-Pad79)
- U7 pad 80: /Block Diagram/Controller/MCU GPIO/PD11 -> unconnected-(U7B-PD11-Pad80)
- U7 pad 81: /Block Diagram/Controller/MCU GPIO/PD12 -> unconnected-(U7B-PD12-Pad81)
- U7 pad 82: /Block Diagram/Controller/MCU GPIO/PD13 -> unconnected-(U7B-PD13-Pad82)
- U7 pad 85: /Block Diagram/Controller/MCU GPIO/PD14 -> unconnected-(U7B-PD14-Pad85)
- U7 pad 86: /Block Diagram/Controller/MCU GPIO/PD15 -> unconnected-(U7B-PD15-Pad86)
- U7 pad 87: /Block Diagram/Controller/MCU GPIO/PG2 -> unconnected-(U7B-PG2-Pad87)
- U7 pad 88: /Block Diagram/Controller/MCU GPIO/PG3 -> unconnected-(U7B-PG3-Pad88)
- U7 pad 89: /Block Diagram/Controller/MCU GPIO/PG4 -> unconnected-(U7B-PG4-Pad89)
- U7 pad 90: /Block Diagram/Controller/MCU GPIO/PG5 -> unconnected-(U7B-PG5-Pad90)
- U7 pad 91: /Block Diagram/Controller/MCU GPIO/PG6 -> unconnected-(U7B-PG6-Pad91)
- U7 pad 92: /Block Diagram/Controller/MCU GPIO/PG7 -> unconnected-(U7B-PG7-Pad92)
- U7 pad 93: /Block Diagram/Controller/MCU GPIO/PG8 -> unconnected-(U7B-PG8-Pad93)
- U7 pad 96: /Block Diagram/Controller/MCU GPIO/PC6 -> unconnected-(U7A-PC6-Pad96)
- U7 pad 97: /Block Diagram/Controller/MCU GPIO/PC7 -> unconnected-(U7A-PC7-Pad97)
- U7 pad 98: /Block Diagram/Controller/MCU GPIO/PC8 -> unconnected-(U7A-PC8-Pad98)
Routing:
- net Net-(U7A-PA8): track 29.9 -> 11.8 mm
- net /Block Diagram/+5V0: track 133.5 -> 115.9 mm, vias 2 -> 5
- net /Block Diagram/+3V3: track 95.4 -> 83.2 mm, vias 3 -> 8
- net /Block Diagram/Communication/RMII_TX_EN: track 30.4 -> 41.2 mm
- net /Block Diagram/Communication/RMII_CRS_DV: track 30.0 -> 38.1 mm
- net /Block Diagram/Communication/RMII_RXD1: track 31.2 -> 38.1 mm
- net /Block Diagram/Communication/RMII_TXD0: track 32.0 -> 37.8 mm
- net /Block Diagram/Communication/RMII_RXD0: track 32.8 -> 38.1 mm
- net /Block Diagram/Communication/RMII_TXD1: track 33.7 -> 38.1 mm
- net /Block Diagram/Controller/NRST: track 122.6 -> 126.8 mm
- net /Block Diagram/Communication/+3V3V: track 74.3 -> 70.4 mm, vias 6 -> 8
- net V_BUS: track 106.0 -> 109.7 mm, vias 2 -> 3
- net Net-(U10-RXD0/MODE0): track 5.19 -> 7.42 mm
- net /Block Diagram/ADC/+REF_RTD2: track 34.6 -> 36.1 mm
- net /Block Diagram/ADC/+A0: track 34.0 -> 32.7 mm
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- added copper zone on B.Cu, net /Block Diagram/+3V3
- added copper zone on B.Cu, net /Block Diagram/+5V0
- added copper zone on F.Cu, net /Block Diagram/+5V0
- added copper zone on B.Cu, net V_BUS
