File: cryonano-nano-stage/cryonano-nano-stage.kicad_pcb (KiCad board)
At the start: 4 copper layers, 100 x 75 mm, 198 parts, among them J1 JST-B3B-XH-AM, J2 JST-B2B-XH-AM, J3 JST-B2B-XH-AM, J5 JST-B3B-XH-AM, J6 RJ45_Hanrun_HR911105A_Horizon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, J8 Conn_ST_STDC14, J9 USB4930-00-A, Q1 PMV100EPAR, SW1 BOOT, SW2 RESET, U1 AD7124-8BCPZ-RL7, U10 LAN8742A, U2 SRDA3.3-4BTG, U3 TLP2735(TP,E(O, U4 AP7363-33D-13, U5 ECMF02-2AMX6, U6 LP5907MFX-3.3_NOPB, U7 STM32H753ZITx, U8 1EDN7550BXTSA1, Y1 12MHz, Y2 32.768kHz, Y3 25.0MHz

Commit message: release candidate
Parts:
- added R101: 0R, Resistor_SMD:R_0805_2012Metric_Pad1.20x1.40mm_HandSolder, B.Cu at (111.3, 126.9)
- added R102: 0R, Resistor_SMD:R_0805_2012Metric_Pad1.20x1.40mm_HandSolder, B.Cu at (128.8, 121.4)
- moved TP1 1.10 mm to (97.0, 117.1)
Connections:
- net Net-(U8-OUT_SNK) renamed /Block Diagram/Heater Drive/G_SINK
- net Net-(U8-OUT_SRC) renamed /Block Diagram/Heater Drive/G_SRC
- net Net-(U8-VDD) renamed /Block Diagram/Heater Drive/DRV_VDD
Routing:
- net Net-(R101-Pad2): track 2.58 -> 7.54 mm, vias 0 -> 1
- net /Block Diagram/ADC/+REF_RTD1: track 33.5 -> 29.8 mm
- net /Block Diagram/+5V0: track 113.1 -> 115.5 mm
- net Net-(U8-IN+): track 5.82 -> 8.07 mm
- net Net-(R102-Pad2): track 2.40 -> 4.40 mm, vias 0 -> 1
- net /Block Diagram/ADC/+REF_RTD2: track 36.3 -> 38.3 mm
- net /Block Diagram/+3V3: track 94.4 -> 92.7 mm
- net /Block Diagram/ADC/-REF_RTD1: track 57.6 -> 56.2 mm
- net /Block Diagram/ADC/REFIOUT: track 14.9 -> 16.1 mm
- net /Block Diagram/ADC/A+3V3: track 71.7 -> 72.8 mm
- net /Block Diagram/ADC/-A1: track 17.4 -> 18.4 mm
- net V_BUS: track 109.3 -> 108.8 mm
- net GND: vias 308 -> 303
