File: cryonano-nano-stage/adc.kicad_sch (KiCad schematic)
At the start: 20 parts, among them U1 AD7124-8BCPZ-RL7, U6 LP5907MFX-3.3_NOPB

Commit message: drc ok, review schematic
Parts:
- added C60: 100n, Capacitor_SMD:C_0603_1608Metric, symbol Device:C_Small
Connections:
- net GND: now also C60.2
- net REFVOUT: now also C60.1

Commit message: release candidate
Parts:
- R77, R78, R79, R80, R81, R82, R83, R84, R85: Order No. 0603/120mW -> 0603, 120mW
