File: cryonano-nano-stage/block-diagram.kicad_sch (KiCad schematic)
At the start: 10 parts, among them J1 24VDC IN, J2 JST-B2B-XH-AM, J3 JST-B2B-XH-AM, J5 JST-B3B-XH-AM

Commit message: sch improved
Connections:
- net Heater Drive/SW_D: now also J5.1; no longer J5.3
- net Heater Drive/SW_G: now also J5.3; no longer J5.2
- net Heater Drive/SW_S: now also J5.2; no longer J5.1
Other:
- sheet ADC ports: added A0+, A0-, A1+, A1-; removed none
- sheet Interface ports: added EQ1+, EQ1-, EQ2+, EQ2-; removed none

Commit message: sch improved
Parts:
- added R88, R89: 0R, Resistor_SMD:R_0805_2012Metric, symbol Device:R_Small
Connections:
- new net ADC/+3V3OUT: R88.1, R89.1
- new net ADC/REFIOUT: R89.2
- new net ADC/REFVOUT: R88.2
Other:
- sheet ADC ports: added +3V3OUT, 0V0OUT, REFIOUT, REFVOUT; removed none
- sheet Communication ports: added ID, VBUS_SENSE; removed none
- sheet Controller ports: added ID, VBUS_SENSE; removed +5V0IN
- sheet Interface ports: added EXCITATION, REF0; removed +5V0IN, 0V0IN

Commit message: pcb drc ok. 68 ohm matching pending
Parts:
- J1, J5: Arrow Part Number B3B-XH-AM(LF)(SN) -> (none); Arrow Price/Stock https://www.arrow.com/en/products/b3b-xh-a-m-lf-sn/jst-manu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 -> (none); Manufacturer_Name JST (JAPAN SOLDERLESS TERMINALS) -> (none); Manufacturer_Part_Number B3B-XH-AM(LF)(SN) -> (none); Mouser Part Number 306-B3BXHAMLFSNP -> (none); Mouser Price/Stock https://www.mouser.co.uk/ProductDetail/JST-Commercial/B3B-X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 -> (none)
- J2, J3: footprint B2BXHAMLFSN -> footprints:B2BXHAMLFSN; Arrow Part Number B2B-XH-AM(LF)(SN) -> (none); Arrow Price/Stock https://www.arrow.com/en/products/b2b-xh-am-lf-sn/jst-manuf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 -> (none); Manufacturer_Name JST (JAPAN SOLDERLESS TERMINALS) -> (none); Manufacturer_Part_Number B2B-XH-AM(LF)(SN) -> (none); Mouser Part Number 306-B2B-XH-AMLFSNP -> (none); Mouser Price/Stock https://www.mouser.co.uk/ProductDetail/JST-Commercial/B2B-X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 -> (none)
Other:
- sheet ADC ports: added +A0, +A1, +REF_RTD1, +REF_RTD2, -A0, -A1, -REF_RTD1, -REF_RTD2; removed A0+, A0-, A1+, A1-, RTD1_REF+, RTD1_REF-, RTD2_REF+, RTD2_REF-
- sheet Interface ports: added +EQ1, +EQ2, +REF_RTD1, +REF_RTD2, -EQ1, -EQ2, -REF_RTD1, -REF_RTD2, REF_RET; removed EQ1+, EQ1-, EQ2+, EQ2-, REF0, RTD1_REF+, RTD1_REF-, RTD2_REF+, RTD2_REF-

Commit message: drc no error, only warnings
Parts:
- R88, R89: footprint Resistor_SMD:R_0805_2012Metric -> Resistor_SMD:R_0805_2012Metric_Pad1.20x1.40mm_HandSolder
Changed lines of the file:
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@@
 			)
 		)
-		(property "Footprint" "Resistor_SMD:R_0805_2012Metric"
+		(property "Footprint" "Resistor_SMD:R_0805_2012Metric_Pad1.20x1.40mm_HandSolder"
 			(at 220.98 71.12 0)
 			(hide yes)
@@
 			)
 		)
-		(property "Footprint" "Resistor_SMD:R_0805_2012Metric"
+		(property "Footprint" "Resistor_SMD:R_0805_2012Metric_Pad1.20x1.40mm_HandSolder"
 			(at 220.98 68.58 0)
 			(hide yes)

Commit message: bom adjusted
Parts:
- H1, H2, H3, H4, H5, H6: Order No. (none) -> N.A.
- J1: value 24VDC IN -> JST-B3B-XH-AM; Order No. (none) -> JST-B3B-XH-AM
- J2, J3: Order No. (none) -> JST-B2B-XH-AM
- J5: Order No. (none) -> JST-B3B-XH-AM
- R88, R89: Order No. (none) -> 0805/250mW
Changed lines of the file:
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@@
 			)
 		)
+		(property "Order No." "N.A."
+			(at 48.26 158.75 0)
+			(hide yes)
+			(show_name no)
+			(do_not_autoplace no)
+			(effects
+				(font
+					(size 1.27 1.27)
+				)
+			)
+		)
 		(instances
 			(project "cryonano-nano-stage"
@@
 			)
 		)
+		(property "Order No." "N.A."
+			(at 25.4 158.75 0)
+			(hide yes)
+			(show_name no)
+			(do_not_autoplace no)
+			(effects
+				(font
+					(size 1.27 1.27)
+				)
+			)
+		)
 		(instances
 			(project "cryonano-nano-stage"
@@
 			)
 		)
+		(property "Order No." "N.A."
+			(at 48.26 165.1 0)
+			(hide yes)
+			(show_name no)
+			(do_not_autoplace no)
+			(effects
+				(font
+					(size 1.27 1.27)
+				)
+			)
+		)
 		(instances
 			(project "cryonano-nano-stage"
@@
 			)
 		)
+		(property "Order No." "N.A."
+			(at 25.4 152.4 0)
+			(hide yes)
+			(show_name no)
+			(do_not_autoplace no)
+			(effects
+				(font
+					(size 1.27 1.27)
+				)
+			)
+		)
 		(instances
 			(project "cryonano-nano-stage"
@@
 			)
 		)
-		(property "Order No." ""
+		(property "Order No." "0805/250mW"
 			(at 220.98 71.12 0)
 			(hide yes)
@@
 			)
 		)
-		(property "Value" "24VDC IN"
+		(property "Value" "JST-B3B-XH-AM"
 			(at 27.178 91.186 0)
 			(show_name no)
@@
 			)
 		)
+		(property "Order No." "JST-B3B-XH-AM"
+			(at 30.48 81.28 0)
+			(hide yes)
+			(show_name no)
+			(do_not_autoplace no)
+			(effects
+				(font
+					(size 1.27 1.27)
+				)
+			)
+		)
 		(pin "1"
 		)
@@
 			)
 		)
+		(property "Order No." "JST-B3B-XH-AM"
+			(at 185.42 125.73 0)
+			(hide yes)
+			(show_name no)
+			(do_not_autoplace no)
+			(effects
+				(font
+					(size 1.27 1.27)
+				)
+			)
+		)
 		(pin "1"
 		)
@@
 			)
 		)
+		(property "Order No." "N.A."
+			(at 48.26 152.4 0)
+			(hide yes)
+			(show_name no)
+			(do_not_autoplace no)
+			(effects
+				(font
+					(size 1.27 1.27)
+				)
+			)
+		)
 		(instances
 			(project "cryonano-nano-stage"
@@
 			)
 		)
-		(property "Order No." ""
+		(property "Order No." "0805/250mW"
 			(at 220.98 68.58 0)
 			(hide yes)
@@
 			)
 		)
+		(property "Order No." "N.A."
+			(at 25.4 165.1 0)
+			(hide yes)
+			(show_name no)
+			(do_not_autoplace no)
+			(effects
+				(font
+					(size 1.27 1.27)
+				)
+			)
+		)
 		(instances
 			(project "cryonano-nano-stage"
@@
 			)
 		)
+		(property "Order No." "JST-B2B-XH-AM"
+			(at 257.81 76.2 0)
+			(hide yes)
+			(show_name no)
+			(do_not_autoplace no)
+			(effects
+				(font
+					(size 1.27 1.27)
+				)
+			)
+		)
 		(pin "1"
 		)
@@
 			(at 257.81 93.98 0)
 			(hide yes)
+			(show_name no)
+			(do_not_autoplace no)
+			(effects
+				(font
+					(size 1.27 1.27)
+				)
+			)
+		)
+		(property "Order No." "JST-B2B-XH-AM"
+			(at 257.81 93.98 0)
+			(hide yes)

Commit message: drc ok, review schematic
Parts:
- added R95: 0R, Resistor_SMD:R_0805_2012Metric_Pad1.20x1.40mm_HandSolder, symbol Device:R_Small
Connections:
- net ADC/+3V3OUT: now also R95.2; no longer R88.1, R89.1
- net Heater Drive/SW_D renamed PSW_D
- net Heater Drive/SW_G renamed PSW_S
- net Heater Drive/SW_S renamed PSW_G
- new net Interface/EXCITATION: R88.1, R89.1, R95.1

Commit message: drc ok. chip level review pending
Other:
- sheet Communication ports: added none; removed ID
- sheet Controller ports: added none; removed ID
Changed lines of the file:
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@@
 	(wire
 		(pts
-			(xy 83.82 104.14) (xy 83.82 114.3)
-		)
-		(stroke
-			(width 0)
-			(type default)
-		)
-	)
-	(wire
-		(pts
 			(xy 53.34 104.14) (xy 53.34 114.3)
 		)
@@
 			)
 		)
-		(pin "ID" input
-			(at 83.82 114.3 90)
-			(effects
-				(font
-					(size 1.27 1.27)
-				)
-				(justify right)
-			)
-		)
 		(pin "VBUS_SENSE" output
 			(at 86.36 114.3 90)
@@
 				)
 				(justify left)
-			)
-		)
-		(pin "ID" input
-			(at 83.82 104.14 270)
-			(effects
-				(font
-					(size 1.27 1.27)
-				)
-				(justify left)
