File: cryonano-nano-stage/block-diagram.kicad_sch (KiCad schematic)
At the start: 13 parts, among them J1 JST-B3B-XH-AM, J2 JST-B2B-XH-AM, J3 JST-B2B-XH-AM, J5 JST-B3B-XH-AM

Commit message: release candidate
Parts:
- R88, R89, R95: Order No. 0805/250mW -> 0805, 250mW
