File: cryonano-nano-stage/communication.kicad_sch (KiCad schematic)
At the start: 40 parts, among them J6 RJ45_Hanrun_HR911105A_Horizon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, J7 10118194-0001LF, U10 LAN8742A, U5 ECMF02-2AMX6, U9 USBLC6-4SC6, Y3 25.0MHz

Commit message: sch improved
Parts:
- U10: footprint Package_DFN_QFN:VQFN-24-1EP_4x4mm_P0.5mm_EP2.5x2.5mm_ThermalVias -> footprints:VQFN-24-1EP_4x4mm_P0.5mm_EP2.5x2.5mm_ThermalVias

Commit message: sch improved
Parts:
- removed R68: 0R, Resistor_SMD:R_0603_1608Metric, symbol Device:R_Small
- removed U9: USBLC6-4SC6, Package_TO_SOT_SMD:SOT-23-6, symbol Power_Protection:USBLC6-4SC6
- added C10: 10u, Capacitor_SMD:C_0805_2012Metric, symbol Device:C_Small
- added C32: 100n, Capacitor_SMD:C_0603_1608Metric, symbol Device:C_Small
- added D5: ESD9X5.0ST5G, SODFL1006X40N, symbol symbols:ESD9X5.0ST5G
- added IC1: KSZ8081MLXCA-TR, QFP50P900X900X160-48N, symbol Samacsys:KSZ8081MLXCA-TR
- added J9: USB4930-00-A, footprints:USB4930-00-A, symbol symbols:USB4930-00-A
- added R76, R90: 5.1k, Resistor_SMD:R_0603_1608Metric, symbol Device:R_Small
- added R87: 10k, Resistor_SMD:R_0603_1608Metric, symbol Device:R_Small
- added U2: NUP4106DR2G, SOIC127P600X175-8N, symbol symbols:NUP4106DR2G
- C31, C38: value 100n -> 22n
- J7: now not fitted; now left out of the parts list
Connections:
- net +3V3V: now also C31.1, C38.1, J6.4 (TCT), J6.5 (RCT), C32.1, U2.2 (REF_1_1), U2.3 (REF_1_2)
- net D+: now also U5.5 (D-_out), J9.A6 (DP1), J9.B6 (DP2); no longer J7.3 (D+), U5.6 (D+_out)
- net D-: now also U5.6 (D+_out), J9.A7 (DN1), J9.B7 (DN2); no longer J7.2 (D-), U5.5 (D-_out)
- net DM: now also U5.1 (D+_in); no longer U5.2 (D-_in)
- net DP: now also U5.2 (D-_in); no longer U5.1 (D+_in)
- net GND: now also C2.1, C10.2, C32.2, D5.2 (A), J9.A1 (GND), J9.A12 (GND), J9.B1 (GND), J9.B12 (GND), R76.2, R87.1, R90.2, U2.5 (GND_1), U2.8 (GND_2); no longer C2.2, J7.5 (GND)
- net GND_SHIELD: now also J6.8; no longer J6.SH
- net LED2: now also R87.2
- net RD_N: now also U10.23 (RXP), U2.1 (I/O_1); no longer U10.22 (RXN)
- net TD_N: now also U10.21 (TXP), U2.6 (I/O_3); no longer U10.20 (TXN)
- net TD_P: now also U10.20 (TXN), U2.4 (I/O_2); no longer U10.21 (TXP)
- net V_BUS: now also C2.2, C10.1; no longer C2.1
- net at C35.1: now also J6.SH; no longer J6.8
- net at C24.2, Y3.1: now also U10.5 (XTAL1/CLKIN)
- net PD_P renamed RD_P
- net RD_P: now also U10.22 (RXN), U2.7 (I/O_4); no longer U10.23 (RXP)
- net VCC_USB: no longer names the net of J7.1 (VCC)
- net VCC_USB: no longer FB8.1
- new net: J9.A5 (CC1), R76.1
- new net: J9.B5 (CC2), R90.1
- new net: FB7.2, J9.17 (SHELL), J9.18 (SHELL), J9.19 (SHELL), J9.20 (SHELL)
- new net VBUS_SENSE: D5.1 (K), FB8.1, J9.A4 (VBUS), J9.A9 (VBUS), J9.B4 (VBUS), J9.B9 (VBUS)
- now unconnected: J7.MH1, J7.MH2, J7.MH3, J7.MH4, J7.MP1, J7.MP2
- no-connect marks 1 -> 2
Other:
- moved on the sheet: C2, C24, C25, C26, C30, C31, C35, C38, FB7, FB8, J6, R57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

Commit message: pcb drc ok. 68 ohm matching pending
Parts:
- C10, C13: footprint Capacitor_SMD:C_0805_2012Metric -> Capacitor_SMD:C_1206_3216Metric; Manufacturer (none) -> KEMET; Order No. (none) -> C1206C106K4RACTU; Unit Price 10 (none) -> 13.5
- C19, C22, C23, C32: Manufacturer (none) -> KEMET; Order No. (none) -> C0603C104K5RAC7411; Tolerence 10% -> (none); Unit Price 10 (none) -> 2.5
- C2: Manufacturer TAIYO YUDEN -> KEMET; Order No. (none) -> C0603C104K5RAC7411; Tolerence 10% -> (none); Unit Price 10 (none) -> 2.5
- C24, C25: value 5.6p -> 8p; Manufacturer (none) -> YAGEO; Order No. (none) -> CC0603DRNPO9BN8R0; Unit Price 10 (none) -> 4
- C26: Manufacturer (none) -> KEMET; Order No. (none) -> C0603C471J5GACTU
- C30: Manufacturer (none) -> KEMET; Order No. (none) -> C0603C105K4RACTU; Unit Price 10 (none) -> 3
- C31, C38: Manufacturer (none) -> KEMET; Order No. (none) -> C0603C223K1RACTU; Unit Price 10 (none) -> 2.1; Voltage 16V -> 50V
- C35: Manufacturer (none) -> KEMET; Order No. (none) -> C0603C102K5RACTU; Unit Price 10 (none) -> 1.2; Voltage 16V -> 50V
- D5: footprint SODFL1006X40N -> footprints:SODFL1006X40N; Arrow Part Number ESD9X5.0ST5G -> (none); Arrow Price/Stock https://www.arrow.com/en/products/esd9x5.0st5g/on-semicondu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 -> (none); Manufacturer_Name onsemi -> (none); Manufacturer_Part_Number ESD9X5.0ST5G -> (none); Mouser Part Number 863-ESD9X5.0ST5G -> (none); Mouser Price/Stock https://www.mouser.co.uk/ProductDetail/onsemi/ESD9X5.0ST5G?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 -> (none)
- IC1: footprint QFP50P900X900X160-48N -> footprints:QFP50P900X900X160-48N; Arrow Part Number KSZ8081MLXCA-TR -> (none); Arrow Price/Stock https://www.arrow.com/en/products/ksz8081mlxca-tr/microchip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 -> (none); Manufacturer_Name Microchip -> (none); Manufacturer_Part_Number KSZ8081MLXCA-TR -> (none); Mouser Part Number 998-KSZ8081MLXCATR -> (none); Mouser Price/Stock https://www.mouser.co.uk/ProductDetail/Microchip-Technology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 -> (none)
- U2: footprint SOIC127P600X175-8N -> footprints:SOIC127P600X175-8N; Manufacturer_Name onsemi -> (none); Manufacturer_Part_Number NUP4106DR2G -> (none); Mouser Part Number 863-NUP4106DR2G -> (none); Mouser Price/Stock https://www.mouser.co.uk/ProductDetail/onsemi/NUP4106DR2G?q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 -> (none)
Connections:
- net D+: now also U5.6 (D+_out); no longer U5.5 (D-_out)
- net D-: now also U5.5 (D-_out); no longer U5.6 (D+_out)
- net DM: now also U5.2 (D-_in); no longer U5.1 (D+_in)
- net DP: now also U5.1 (D+_in); no longer U5.2 (D-_in)
- net XTAL1: now reaches C24.2, U10.5 (XTAL1/CLKIN), Y3.1
- net XTAL2: now reaches C25.2, U10.4 (XTAL2), Y3.3
- net RD_N renamed ETH_RD_N
- net RD_P renamed ETH_RD_P
- net TD_N renamed ETH_TD_N
- net TD_P renamed ETH_TD_P

Commit message: bom adjusted
Parts:
- removed D5: ESD9X5.0ST5G, footprints:SODFL1006X40N, symbol symbols:ESD9X5.0ST5G
- removed U2: NUP4106DR2G, footprints:SOIC127P600X175-8N, symbol symbols:NUP4106DR2G
- added D5: SMF5V0A-M3-08, Diode_SMD:D_SMF, symbol symbols:SMF5V0A-M3-08
- added U2: SRDA3.3-4BTG, Package_SO:SOIC-8_3.9x4.9mm_P1.27mm, symbol symbols:SRDA3.3-4BTG
- FB7, FB8: Order No. BLM21PG221SN1D -> BLM21PG221BH1D
- J6: Order No. (none) -> HR911105A
- J9: Order No. (none) -> USB4930-00-A
- R57, R58, R59, R60, R61, R62, R63, R64, R65, R66, R67, R69, R70, R71, R72, R73, R74, R75, R76, R87, R90: Order No. (none) -> 0603/120mW
- U10: Order No. (none) -> LAN8742A
Connections:
- net +3V3V: now also U2.2 (REF_1_1), U2.3 (REF_1_2)
- net ETH_RD_N: now also U2.1 (I/O_1)
- net ETH_RD_P: now also U2.7 (I/O_4)
- net ETH_TD_N: now also U2.6 (I/O_3)
- net ETH_TD_P: now also U2.4 (I/O_2)
- net GND: now also D5.1 (A), U2.5 (GND_1), U2.8 (GND_2)
- net VBUS_SENSE: now also D5.2 (C)

Commit message: release candidate
Parts:
- IC1: Order No. (none) -> KSZ8081MLXCA-TR
- R57, R58, R59, R60, R61, R62, R63, R64, R65, R66, R67, R69, R70, R71, R72, R73, R74, R75, R76, R87, R90: Order No. 0603/120mW -> 0603, 120mW
