File: cryonano-nano-stage/heater-controller.kicad_sch (KiCad schematic)
At the start: 21 parts, among them U3 TLP2735(TP,E(O, U8 1EDN7550BXTSA1

Commit message: sch reviewed
Parts:
- added C63: 680p, Capacitor_SMD:C_0603_1608Metric, symbol Device:C_Small
- added D9: SMBJE36CAH, Diode_SMD:D_SMB, symbol symbols:SMBJE36CAH
- added R100: 6R2, Resistor_SMD:R_2010_5025Metric, symbol Device:R_Small
- added R29: 2.7k, Resistor_SMD:R_0805_2012Metric, symbol Device:R_Small
- added R99: 56R, Resistor_SMD:R_2010_5025Metric, symbol Device:R_Small
- C62: value 100n -> 680p; Manufacturer KEMET -> (none); Order No. C0603C104K5RAC7411 -> (none); Unit Price 10 2.5 -> (none); Voltage 16V -> 50V
Connections:
- net +15V0: now also R29.2
- net SW_D: now also D9.2
- net SW_S: now also R100.1, R29.1, R99.1
- net at R39.1: now also U8.5 (OUT_SRC); no longer U8.6 (OUT_SNK)
- net at R37.1: now also U8.6 (OUT_SNK); no longer U8.5 (OUT_SRC)
- new net: C63.1, D9.1, R99.2
- new net: C63.2, R100.2
- no-connect marks 1 -> 0
Other:
- note added: "Drain snubber."
- note added: "Gate snubber."
- note added: "Note: 1. MOSFET V_DS >= 100 V, V_GS >= 20 V 2. Drain snubber section is to be populated only if the switch has no local snubber."
- moved on the sheet: C61, FB6, R27, R28, R37, R39, R97, R98, U8, Z2

Commit message: release candidate
Parts:
- C39: Order No. (none) -> 50 V, 0805, X7R
- C62, C63: Order No. (none) -> 0603, C0G/NP0
- D9: Order No. (none) -> SMBJE36CAH
- R100, R99: Order No. (none) -> 2010, 2W
- R27, R28, R40: Order No. 0603/120mW -> 0603, 120mW
- R29: Order No. 0805/225mW -> 0805, 225mW
- R97, R98: Order No. (none) -> 0603, 120mW
- U3: Order No. (none) -> TLP2735(TP,E(O
- U8: Arrow Part Number 1EDN7550BXTSA1 -> (none); Arrow Price/Stock https://www.arrow.com/en/products/1edn7550bxtsa1/infineon-t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 -> (none); Manufacturer_Name Infineon -> (none); Manufacturer_Part_Number 1EDN7550BXTSA1 -> (none); Mouser Part Number 726-1EDN7550BXTSA1 -> (none); Mouser Price/Stock https://www.mouser.co.uk/ProductDetail/Infineon-Technologie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 -> (none); Order No. (none) -> 1EDN7550BXTSA1
Connections:
- net DRV_VDD: now reaches C61.1, FB6.2, U8.4 (VDD)
- net G_SRC: now reaches R39.1, U8.5 (OUT_SRC)
- net G_SINK: now reaches R37.1, U8.6 (OUT_SNK)
Other:
- moved on the sheet: R27, R37, R39, Z2
